File: main_hw/SUMEC_MK_IV_Pro/MCU.kicad_sch (KiCad schematic)
At the start: 28 parts, among them J2 USB_TypeC, SW2 SW_Push, SW3 SW_Push, SW4 SW_Push, SW5 SW_Push, U2 ESP32-S3-WROOM-1, U3 USBLC6-2SC6

Commit message: Schematic update
Parts:
- removed C19, C22, C23, C24: 100nF, Capacitor_SMD:C_0805_2012Metric_Pad1.18x1.45mm_HandSolder, symbol Device:C
- removed D3, D4, D5, D6, D7: LED, LED_SMD:LED_0805_2012Metric_Pad1.15x1.40mm_HandSolder, symbol Device:LED
- removed F1: Polyfuse/50R, Fuse:Fuse_0805_2012Metric, symbol Device:Polyfuse
- removed J2: USB_TypeC, sumec_brd:HRO_TYPE-C-31-M-12, symbol sumec_sch_lib:USB_TypeC
- removed R12: 100k, Resistor_SMD:R_0805_2012Metric_Pad1.20x1.40mm_HandSolder, symbol Device:R
- removed R13, R14: 15R, Resistor_SMD:R_0805_2012Metric_Pad1.20x1.40mm_HandSolder, symbol Device:R
- removed R15: 10k, Resistor_SMD:R_0805_2012Metric_Pad1.20x1.40mm_HandSolder, symbol Device:R
- removed R16: 560R, Resistor_SMD:R_0805_2012Metric_Pad1.20x1.40mm_HandSolder, symbol Device:R
- removed R17: 200R, Resistor_SMD:R_0805_2012Metric_Pad1.20x1.40mm_HandSolder, symbol Device:R
- removed R18, R19, R20: 100R, Resistor_SMD:R_0805_2012Metric_Pad1.20x1.40mm_HandSolder, symbol Device:R
- removed SW2, SW3, SW4, SW5: SW_Push, sumec_brd:SW_SPST_EVQPE1, symbol Switch:SW_Push
- removed U3: USBLC6-2SC6, Package_TO_SOT_SMD:TSOT-23-6_HandSoldering, symbol sumec_library:USBLC6-2SC6
Connections:
- no-connect marks 9 -> 5
Other:
- note removed: "BOOT"
- note removed: "Battery power"
- note removed: "Buttons for BOOT and ENABLE functions. If the device does not support the auto download mode, you need to get into the download mode manually. To do so, press and hold the BOOT button and then press the RESET button once. After that release the BOOT button."
- note removed: "EN=RESET, BOOT=bootloader mode Enable (EN) is the 3.3V regulator's enable pin. It's pulled up, so connect to ground to disable the 3.3V regulator. This means that you can use this pin connected to a pushbutton to restart your ESP32, for example."
- note removed: "ENABLE"
- note removed: "ESD PROTECTION"
- note removed: "GPIO USB 20 D+ (green) 19 D- (white) GND GND (black) VBUS +5V (red)"
- note removed: "LED SIGNALISATION"
- note removed: "PUSH BUTTONS"
- note removed: "Status LED1"
- note removed: "Status LED2"
- note removed: "Status LED3"
- note removed: "USB"
- note removed: "USB CONNECTOR"
- note removed: "USB Type-C Connector Data transfer USB connector connected to ESP32 using CDC method"
- note removed: "VBUS Power"
- moved on the sheet: C20, C21, U2
