File: main_hw/SUMEC_MK_IV_Pro/CONNECTIVITY.kicad_sch (KiCad schematic)
At the start: 17 parts, among them J10 Conn_01x03_Pin, J11 Conn_01x03_Pin, J12 Conn_01x06_Socket, J13 Conn_01x03_Pin, J14 Conn_01x06_Socket, J3 Conn_01x06_Pin, J4 Conn_01x06_Pin, J5 Conn_01x03_Pin, J6 Conn_01x03_Pin, J7 Conn_01x06_Pin, J8 Conn_01x04_Pin, J9 Conn_01x03_Pin, U4 TSOP382xx

Commit message: Schematic update
Parts:
- removed C25, C26: 10uF, Capacitor_Tantalum_SMD:CP_EIA-3216-18_Kemet-A_Pad1.58x1.35mm_HandSolder, symbol Device:C_Polarized
- removed J10, J11, J13, J5, J6, J9: Conn_01x03_Pin, Connector_Molex:Molex_PicoBlade_53398-0371_1x03-1MP_P1.25mm_Vertical, symbol Connector:Conn_01x03_Pin
- removed J12, J14: Conn_01x06_Socket, Connector_JST:JST_SH_BM06B-SRSS-TB_1x06-1MP_P1.00mm_Vertical, symbol Connector:Conn_01x06_Socket
- removed J3, J4, J7: Conn_01x06_Pin, Connector_Molex:Molex_PicoBlade_53398-0671_1x06-1MP_P1.25mm_Vertical, symbol Connector:Conn_01x06_Pin
- removed J8: Conn_01x04_Pin, Connector_Molex:Molex_PicoBlade_53398-0471_1x04-1MP_P1.25mm_Vertical, symbol Connector:Conn_01x04_Pin
- removed R21: 10k, Resistor_SMD:R_0805_2012Metric_Pad1.20x1.40mm_HandSolder, symbol Device:R
- removed R22: 100R, Resistor_SMD:R_0805_2012Metric_Pad1.20x1.40mm_HandSolder, symbol Device:R
- removed U4: TSOP382xx, sumec_brd:Vishay_TSOP382, symbol Interface_Optical:TSOP382xx
- added C19, C22: 100nF, Capacitor_SMD:C_0805_2012Metric_Pad1.18x1.45mm_HandSolder, symbol Device:C
- added D3, D4, D5, D6, D7: LED, LED_SMD:LED_0805_2012Metric_Pad1.15x1.40mm_HandSolder, symbol Device:LED
- added F1: Polyfuse/50R, Fuse:Fuse_0805_2012Metric, symbol Device:Polyfuse
- added J2: USB_TypeC, sumec_brd:HRO_TYPE-C-31-M-12, symbol sumec_sch_lib:USB_TypeC
- added R12: 100k, Resistor_SMD:R_0805_2012Metric_Pad1.20x1.40mm_HandSolder, symbol Device:R
- added R13, R14: 15R, Resistor_SMD:R_0805_2012Metric_Pad1.20x1.40mm_HandSolder, symbol Device:R
- added R16: 560R, Resistor_SMD:R_0805_2012Metric_Pad1.20x1.40mm_HandSolder, symbol Device:R
- added R17: 200R, Resistor_SMD:R_0805_2012Metric_Pad1.20x1.40mm_HandSolder, symbol Device:R
- added R18, R19, R20: 100R, Resistor_SMD:R_0805_2012Metric_Pad1.20x1.40mm_HandSolder, symbol Device:R
- added U3: USBLC6-2SC6, Package_TO_SOT_SMD:TSOT-23-6_HandSoldering, symbol sumec_library:USBLC6-2SC6
Connections:
- net GND: now also C19.1, C22.2, J2.A1_B12 (GND), J2.B1_A12 (GND), R12.2, R16.2, R17.2, R18.2, R19.2, R20.2, U3.2
- new net: D7.1 (K), R20.1
- new net: D3.1 (K), R16.1
- new net: D4.1 (K), R17.1
- new net: D5.1 (K), R18.1
- new net: R14.2, U3.3
- new net: R13.2, U3.1
- new net: F1.2, J2.A4_B9 (VBUS), J2.B4_A9 (VBUS)
- new net: D6.1 (K), R19.1
- new net +12V: D3.2 (A)
- new net D+: U3.6
- new net D+ IN: J2.A6 (DP1), J2.B6 (DP2), R13.1
- new net D-: U3.4
- new net D- IN: J2.A7 (DN1), J2.B7 (DN2), R14.1
- new net LED_IO_13: D7.2 (A)
- new net LED_IO_14: D6.2 (A)
- new net LED_IO_21: D5.2 (A)
- new net SHLD: C19.2, J2.S1 (SHIELD), J2.S2 (SHIELD), J2.S3 (SHIELD), J2.S4 (SHIELD), R12.1
- new net VBUS 5V: C22.1, D4.2 (A), F1.1, U3.5
- no-connect marks 3 -> 4
Other:
- note added: "Battery power"
- note added: "ESD PROTECTION"
- note added: "GPIO USB 20 D+ (green) 19 D- (white) GND GND (black) VBUS +5V (red)"
- note added: "LED SIGNALISATION"
- note added: "Status LED1"
- note added: "Status LED2"
- note added: "Status LED3"
- note added: "USB"
- note added: "USB CONNECTOR"
- note added: "USB Type-C Connector Data transfer USB connector connected to ESP32 using CDC method"
- note added: "VBUS Power"
- note removed: "( Better manual in -DOCS- )"
- note removed: "6-PIN JST SH-Style male connector VCC 2.7 V to 18 V encoder operating voltage"
- note removed: "DISTANCE MEASURING"
- note removed: "Digital distance sensor - Sharp GP2Y0D810Z0F Sensor detects objects between 2 cm and 10 cm Low when detecting an object, high otherwise. Frequency - 390 Hz Operating voltage 2.7V - 6.2V"
- note removed: "Digital distance sensor - Sharp GP2Y0D810Z0F Sensor detects objects between 2 cm and 10 cm Low when detecting an object, high otherwise. Operating voltage 2.7V - 6.2V"
- note removed: "IR LED Reciver module Operating voltage: 2.7V to 5.5V Frequency: 38kHz"
- note removed: "IR LED Reciver module Operating voltage: 2.7V to 5.5V Frequency: 38kHz High immunity against ambient light. For more than 1 input use - Hexadecimal code Used as a main program starter"
- note removed: "IR MODULE"
- note removed: "LINE SENSORS"
- note removed: "M1"
- note removed: "M2"
- note removed: "MIRRORED"
- note removed: "MOTORS"
- note removed: "Miniature Reflective Object Sensor - QRE1113 IR reflectance sensor is comprised of two parts - an IR emitting LED and an IR sensitive phototransistor. Analog output A 100Ω resistor is placed in series with the LED to limit current. A 10kΩ resistor pulls the output pin high, but when the light from the LED is reflected back onto the phototransistor the output will begin to go lower. 2 front sensor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"
- note removed: "OBJECT DETECTING SENSORS"
- note removed: "POLOLU SENSOR MANUAL"
- note removed: "Pololu Distance Sensor with Pulse Width Output/Digital Output Small lidar based sensor can report presnece/distance of objects up to (TOTAL MAX 200cm-Digital, 300cm - PWM) Distance is chosen by configurating the jumpers with 0R resistors"
- note removed: "SIDE SENSORS"
- note removed: "TF-LUNA MANUAL"
- note removed: "Time-of-Flight(ToF) laser-ranging module - TF-Luna COMMUNICATION PROTOCOL: I²C When pin 5 is connected to ground, TF-Luna enters I2C mode, then its pin 2 is used as SDA data and pin 3 is the SCL clock sending data."

Commit message: Force push
Parts:
- R16: value 560R -> 1000k
- R17: value 200R -> 220R
- R18, R19, R20: value 100R -> 220R
Connections:
- net VBUS 5V: no longer C22.1, F1.1, U3.5
- net D+ IN renamed D_POS_IN
- net D- IN renamed D_NEG_IN
- net LED_IO_13 renamed LED_3
- net LED_IO_14 renamed LED_2
- net LED_IO_21 renamed LED_1
- new net VBUS_5V: C22.1, F1.1, U3.5
Other:
- moved on the sheet: C22, R13, R14, U3
