File: main_hw/SUMEC_MK_IV_Pro/MECHANICS.kicad_sch (KiCad schematic)
At the start: 9 parts

Commit message: Schematic update
Parts:
- added C23, C24: 100nF, Capacitor_SMD:C_0805_2012Metric_Pad1.18x1.45mm_HandSolder, symbol Device:C
- added R15: 10k, Resistor_SMD:R_0805_2012Metric_Pad1.20x1.40mm_HandSolder, symbol Device:R
- added SW2, SW3, SW4, SW5: SW_Push, sumec_brd:SW_SPST_EVQPE1, symbol Switch:SW_Push
Connections:
- net +3V3: now also R15.2, SW3.1, SW4.1
- net GND: now also C23.2, C24.2, SW2.1, SW5.1
- new net BOOT: C24.1, SW5.2
- new net BUTTON_IO_47: SW4.2
- new net BUTTON_IO_48: SW3.2
- new net EN: C23.1, R15.1, SW2.2
Other:
- note added: "BOOT"
- note added: "Buttons for BOOT and ENABLE functions. If the device does not support the auto download mode, you need to get into the download mode manually. To do so, press and hold the BOOT button and then press the RESET button once. After that release the BOOT button."
- note added: "EN=RESET, BOOT=bootloader mode Enable (EN) is the 3.3V regulator's enable pin. It's pulled up, so connect to ground to disable the 3.3V regulator. This means that you can use this pin connected to a pushbutton to restart your ESP32, for example."
- note added: "ENABLE"
- note added: "PUSH BUTTONS"
- moved on the sheet: H1, H2, H3, H4, TP1, TP2, TP3, TP4, TP5
