File: main_hw/SUMEC_MK_IV_Pro/POWER_SUPPLY.kicad_sch (KiCad schematic)
At the start: 25 parts, among them IC1 TPS565242DRLR, J1 XT30PW-M, Q1 Q_PMOS, Q2 Q_PMOS, SW1 SW_DPDT_x2, U1 TPS62133

Commit message: Force push
Connections:
- net VBUS 5V renamed VBUS_5V
- net VOUT 5V renamed VOUT_5V
Changed lines of the file:
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@@
 		)
 	)
-	(global_label "VOUT 5V"
+	(global_label "VOUT_5V"
 		(shape input)
 		(at 72.39 83.82 180)
@@
 		)
 		(property "Intersheetrefs" "${INTERSHEET_REFS}"
-			(at 64.9801 83.82 0)
+			(at 64.7457 83.82 0)
 			(effects
 				(font
@@
 		)
 	)
-	(global_label "VBUS 5V"
+	(global_label "VBUS_5V"
 		(shape input)
 		(at 57.15 95.25 180)
@@
 		)
 		(property "Intersheetrefs" "${INTERSHEET_REFS}"
-			(at 49.5526 95.25 0)
+			(at 49.3181 95.25 0)
 			(effects
 				(font
@@
 		)
 	)
-	(global_label "VOUT 5V"
+	(global_label "VOUT_5V"
 		(shape output)
 		(at 243.84 96.52 0)
@@
 		)
 		(property "Intersheetrefs" "${INTERSHEET_REFS}"
-			(at 251.2499 96.52 0)
+			(at 251.4843 96.52 0)
 			(effects
 				(font
@@
 		)
 	)
-	(global_label "VBUS 5V"
+	(global_label "VBUS_5V"
 		(shape input)
 		(at 91.44 105.41 0)
@@
 		)
 		(property "Intersheetrefs" "${INTERSHEET_REFS}"
-			(at 99.0374 105.41 0)
+			(at 99.2719 105.41 0)
 			(effects
 				(font
