File: main_hw/SUMEC_MK_IV_Pro/SENSORICS.kicad_sch (KiCad schematic)
At the start: 15 parts, among them J10 Conn_01x03_Pin, J11 Conn_01x03_Pin, J13 Conn_01x03_Pin, J3 Conn_01x06_Pin, J4 Conn_01x06_Pin, J5 Conn_01x03_Pin, J6 Conn_01x03_Pin, J7 Conn_01x06_Pin, J8 Conn_01x04_Pin, J9 Conn_01x03_Pin, U4 TSOP382xx

Commit message: Force push
Parts:
- removed U4: TSOP382xx, sumec_brd:Vishay_TSOP382, symbol Interface_Optical:TSOP382xx
- added C?: 100nF, Capacitor_SMD:C_0805_2012Metric_Pad1.18x1.45mm_HandSolder, symbol Device:C
- added J?: Conn_01x03_Pin, Connector_Molex:Molex_PicoBlade_53398-0371_1x03-1MP_P1.25mm_Vertical, symbol Connector:Conn_01x03_Pin
- added U?: BMI088, BMI088:PQFN50P450X300X100-16N, symbol finca_lib:BMI088
Connections:
- net +3V3: now also J?.3 (Pin_3)
- net GND: now also C?.1, J?.1 (Pin_1), U?.10 (SDO2), U?.15 (SDO1), U?.4 (GNDA), U?.6 (GNDIO)
- net SCL: now also U?.8 (SCL/SCK)
- net SDA: now also U?.9 (SDA/SDI)
- net IO05_POL_R renamed POL_R
- net IO15_POL_M renamed POL_M
- net IO16_POL_L renamed POL_L
- net QRE1113 A renamed QRE_R
- net QRE1113 B renamed QRE_L
- net QRE1113 C renamed QRE_BACK
- net SHARP 1 renamed SHARP_L
- net SHARP 2 renamed SHARP_R
- new net +3.3V: C?.2, U?.11 (VDDIO), U?.3 (VDD), U?.7 (PS)
- new net ACCEL_INTERRUPT_1: U?.16 (INT1)
- new net ACCEL_INTERRUPT_2: U?.1 (INT2)
- new net GYRO_INTERRUPT_1: U?.12 (INT3)
- new net GYRO_INTERRUPT_2: U?.13 (INT4)
- new net IR_MODULE: J?.2 (Pin_2)
- no-connect marks 3 -> 6
Other:
- note added: "*The unit price is set for an order quantity of 10 units"
- note added: "1. Q: VDD and VDDIO needs to be a different voltage? Check videos and other schematics. 2. Q: [] 3. Q: [] 4. Q: [] 5. Q: []"
