File: main_hw/SUMEC_MK_IV_Pro/SUMEC_MK_IV_Pro.kicad_sch (KiCad schematic)
At the start: 7 parts, among them J15 39502-1009, J16 39502-1009, U5 TBA2-0511, U6 NCP1117-3.3

Commit message: Schematic update
Parts:
- added J12, J14: Conn_01x06_Socket, Connector_JST:JST_SH_BM06B-SRSS-TB_1x06-1MP_P1.00mm_Vertical, symbol Connector:Conn_01x06_Socket
- added TP10: TestPoint, sumec_graphic:FREEFALL2_IMG, symbol Connector:TestPoint
- added TP11: TestPoint, sumec_graphic:ME_FR_IMG, symbol Connector:TestPoint
- added TP6: TestPoint, sumec_graphic:SPS_LOGO_IMG, symbol Connector:TestPoint
- added TP7: TestPoint, sumec_graphic:SUMEC_LOGO_IMG, symbol Connector:TestPoint
- added TP8: TestPoint, sumec_graphic:ULTRAKILL_IMG, symbol Connector:TestPoint
- added TP9: TestPoint, sumec_graphic:SUMEC_QR_IMG, symbol Connector:TestPoint
Connections:
- net GND: now also J12.1 (Pin_1), J14.1 (Pin_1)
- new net: TP10.1, TP11.1, TP6.1, TP7.1, TP8.1, TP9.1
- new net +3V3: J12.4 (Pin_4), J14.4 (Pin_4)
- new net M1A: J12.6 (Pin_6)
- new net M1B: J12.5 (Pin_5)
- new net M2A: J14.6 (Pin_6)
- new net M2B: J14.5 (Pin_5)
- new net OUT 1A: J12.3 (Pin_3)
- new net OUT 1B: J12.2 (Pin_2)
- new net OUT 2A: J14.3 (Pin_3)
- new net OUT 2B: J14.2 (Pin_2)
- no-connect marks 1 -> 2
Other:
- removed sheet GRAPHICS
- added sheet SENSORICS (SENSORICS.kicad_sch)
- note added: "6-PIN JST SH-Style male connector VCC 2.7 V to 18 V encoder operating voltage"
- note added: "ART"
- note added: "FREEFALL PANEL"
- note added: "M1"
- note added: "M2"
- note added: "ME FR"
- note added: "MOTORS"
- note added: "SPS LOGO"
- note added: "SUMEC LINKTREE"
- note added: "SUMEC LOGO"
- note added: "ULTRAKILL V1"

Commit message: Force push
Parts:
- removed J12, J14: Conn_01x06_Socket, Connector_JST:JST_SH_BM06B-SRSS-TB_1x06-1MP_P1.00mm_Vertical, symbol Connector:Conn_01x06_Socket
Other:
- note added: "1. Q: Gyro+accelometer - possible to add 2. Q: Passive buzzer 3. Q: Left/right silk for sensors and motors 4. Q: External eeprom? FRAM? 5. Q: Add IO pin numbers after the routing is done 6. Q: VBATT voltage read"
- note removed: "1. Q: Gyro+accelometer - possible to add 2. Q: Passive buzzer 3. Q: Left/right silk for sensors and motors 4. Q: [] 5. Q: []"
- note removed: "6-PIN JST SH-Style male connector VCC 2.7 V to 18 V encoder operating voltage"
- note removed: "M1"
- note removed: "M2"
- note removed: "MOTORS"
