File: Hardware/HadesMicro/HadesMicro.kicad_pcb (KiCad board)
At the start: 4 copper layers, 50 x 50 mm, 91 parts

Commit message: HadesMicro and other PCBs with IMUs
Other:
- net class Default removed
