File: main_hw/SUMEC_MK_V/SUMEC_MK_V.kicad_pcb (KiCad board)
At the start: 4 copper layers, 84.8 x 79.1 mm, 112 parts, among them IC1 TPS565242DRLR, IC2 DRV8874PWPR, IC3 DRV8874PWPR, J1 XT30PW-M, J10 Conn_01x03_Pin, J11 Conn_01x03_Pin, J12 Conn_01x03_Pin, J13 Conn_01x03_Pin, J14 Conn_01x03_Pin, J15 Conn_01x03_Pin, J2 Conn_01x06_Socket, J3 Conn_01x06_Socket, J4 USB_TypeC, J5 Conn_01x04_Pin, J6 Conn_01x06_Pin, J7 Conn_01x06_Pin, J8 Conn_01x03_Pin, J9 Conn_01x06_Pin, Q1 Q_PMOS, Q2 Q_PMOS, SW1 SW_DPDT_x2, SW2 SW_Push, SW3 SW_Push, SW4 SW_Push, SW5 SW_Push, U1 INA226, U2 TPS62133, U3 24CW1280T-I/OT, U4 ESP32-S3-WROOM-1, U5 USBLC6-2SC6, U6 BMI088

Commit message: MK V Schematic update
Parts:
- removed the C16 at (98.3, 125.0)
- removed the C17 at (98.3, 128.0)
- removed the C20 at (160.1, 99.3)
- removed the C22 at (160.1, 102.3)
- removed the IC2 at (114.6, 114.9)
- removed R1, R2, R23: 0R, Resistor_SMD:R_0805_2012Metric_Pad1.20x1.40mm_HandSolder
- removed R14: 0R/R-Ipropi, Resistor_SMD:R_0805_2012Metric_Pad1.20x1.40mm_HandSolder
- removed the R15 at (103.1, 127.7)
- removed the R16 at (107.8, 113.0)
- removed R20: 100k, Resistor_SMD:R_0805_2012Metric_Pad1.20x1.40mm_HandSolder
- removed R21, R22: 15R, Resistor_SMD:R_0805_2012Metric_Pad1.20x1.40mm_HandSolder
- added C16: 22nF, Capacitor_SMD:C_0805_2012Metric_Pad1.18x1.45mm_HandSolder, F.Cu at (141.3, 67.1)
- added C16: 22nF, Capacitor_SMD:C_0805_2012Metric_Pad1.18x1.45mm_HandSolder, F.Cu at (150.6, 67.2)
- added C17: 100nF, Capacitor_SMD:C_0805_2012Metric_Pad1.18x1.45mm_HandSolder, B.Cu at (140.2, 67.0)
- added C17: 100nF, Capacitor_SMD:C_0805_2012Metric_Pad1.18x1.45mm_HandSolder, B.Cu at (149.5, 67.0)
- added C20: 100nF, Capacitor_SMD:C_0805_2012Metric_Pad1.18x1.45mm_HandSolder, F.Cu at (146.8, 67.2)
- added C20: 100nF, Capacitor_SMD:C_0805_2012Metric_Pad1.18x1.45mm_HandSolder, F.Cu at (137.5, 67.1)
- added C22: 10uF, Capacitor_Tantalum_SMD:CP_EIA-3216-18_Kemet-A_Pad1.58x1.35mm_HandSolder, F.Cu at (139.3, 69.2)
- added C22: 10uF, Capacitor_Tantalum_SMD:CP_EIA-3216-18_Kemet-A_Pad1.58x1.35mm_HandSolder, F.Cu at (148.6, 69.2)
- added C31: 10uF, Capacitor_Tantalum_SMD:CP_EIA-3216-18_Kemet-A_Pad1.58x1.35mm_HandSolder, B.Cu at (204.3, 66.2)
- added C32: 100nF, Capacitor_SMD:C_0805_2012Metric_Pad1.18x1.45mm_HandSolder, F.Cu at (164.2, 51.5)
- added C33: 10uF, Capacitor_Tantalum_SMD:CP_EIA-3216-18_Kemet-A_Pad1.58x1.35mm_HandSolder, B.Cu at (204.3, 63.0)
- added C34: 100nF, Capacitor_SMD:C_0805_2012Metric_Pad1.18x1.45mm_HandSolder, F.Cu at (164.2, 54.5)
- added IC2: DRV8874PWPR, sumec_brd:DRV8874, F.Cu at (149.3, 62.2)
- added IC2: DRV8874PWPR, sumec_brd:DRV8874, F.Cu at (140.0, 62.2)
- added JP1: SolderJumper_3_Open, Jumper:SolderJumper-3_P2.0mm_Open_TrianglePad1.0x1.5mm, F.Cu at (169.5, 72.2)
- added JP2: SolderJumper_3_Open, Jumper:SolderJumper-3_P2.0mm_Open_TrianglePad1.0x1.5mm, F.Cu at (153.4, 63.0)
- added JP2: SolderJumper_3_Open, Jumper:SolderJumper-3_P2.0mm_Open_TrianglePad1.0x1.5mm, F.Cu at (144.2, 63.0)
- added JP3: SolderJumper_3_Open, Jumper:SolderJumper-3_P2.0mm_Open_TrianglePad1.0x1.5mm, F.Cu at (230.3, 51.0)
- added L3: 3.3uH, Inductor_SMD:L_Vishay_IHLP-1616, F.Cu at (118.7, 66.3)
- added R15: 0R/R-Ipropi, Resistor_SMD:R_0805_2012Metric_Pad1.20x1.40mm_HandSolder, B.Cu at (149.3, 60.1)
- added R15: 0R/R-Ipropi, Resistor_SMD:R_0805_2012Metric_Pad1.20x1.40mm_HandSolder, B.Cu at (140.1, 60.1)
- added R16: 0R/R-Imode, Resistor_SMD:R_0805_2012Metric_Pad1.20x1.40mm_HandSolder, B.Cu at (138.2, 60.1)
- added R16: 0R/R-Imode, Resistor_SMD:R_0805_2012Metric_Pad1.20x1.40mm_HandSolder, B.Cu at (147.4, 60.1)
- added R32: 220R, Resistor_SMD:R_0805_2012Metric_Pad1.20x1.40mm_HandSolder, F.Cu at (19.0, 77.7)
- added R33: 10k, Resistor_SMD:R_0805_2012Metric_Pad1.20x1.40mm_HandSolder, B.Cu at (96.0, 57.0)
- added R34: 10k, Resistor_SMD:R_0805_2012Metric_Pad1.20x1.40mm_HandSolder, F.Cu at (125.8, 30.8)
- added R35: 100R, Resistor_SMD:R_0805_2012Metric_Pad1.20x1.40mm_HandSolder, F.Cu at (125.8, 33.0)
- added U7: BMI088, finca:PQFN50P450X300X100-16N, F.Cu at (168.8, 53.4)
- C12: value 22nF -> 10uF; footprint Capacitor_SMD:C_0805_2012Metric_Pad1.18x1.45mm_HandSolder -> Capacitor_Tantalum_SMD:CP_EIA-3216-18_Kemet-A_Pad1.58x1.35mm_HandSolder
- C14: value 22nF -> 22uF; footprint Capacitor_SMD:C_0805_2012Metric_Pad1.18x1.45mm_HandSolder -> Capacitor_Tantalum_SMD:CP_EIA-2012-12_Kemet-R_Pad1.30x1.05mm_HandSolder
- C15: value 100nF -> 22uF; footprint Capacitor_SMD:C_0805_2012Metric_Pad1.18x1.45mm_HandSolder -> Capacitor_Tantalum_SMD:CP_EIA-2012-12_Kemet-R_Pad1.30x1.05mm_HandSolder
- C18: value 10uF -> 22nF; footprint Capacitor_Tantalum_SMD:CP_EIA-3216-18_Kemet-A_Pad1.58x1.35mm_HandSolder -> Capacitor_SMD:C_0805_2012Metric_Pad1.18x1.45mm_HandSolder
- C19, C21, C27: value 10uF -> 100nF; footprint Capacitor_Tantalum_SMD:CP_EIA-3216-18_Kemet-A_Pad1.58x1.35mm_HandSolder -> Capacitor_SMD:C_0805_2012Metric_Pad1.18x1.45mm_HandSolder
- C23: value 100nF -> 10uF; footprint Capacitor_SMD:C_0805_2012Metric_Pad1.18x1.45mm_HandSolder -> Capacitor_Tantalum_SMD:CP_EIA-3216-18_Kemet-A_Pad1.58x1.35mm_HandSolder
- C25: value 100nF -> 10uF; footprint Capacitor_SMD:C_0805_2012Metric_Pad1.18x1.45mm_HandSolder -> Capacitor_Tantalum_SMD:CP_EIA-3216-18_Kemet-A_Pad1.58x1.35mm_HandSolder; moved to B.Cu
- C26, C30, J1, J10, J11, J12, J14, J15, J2, J3, J5, J8, Q1, R5: moved to B.Cu
- C29: value 10uF -> 100nF; footprint Capacitor_Tantalum_SMD:CP_EIA-3216-18_Kemet-A_Pad1.58x1.35mm_HandSolder -> Capacitor_SMD:C_0805_2012Metric_Pad1.18x1.45mm_HandSolder; moved to B.Cu
- J13: footprint Connector_Molex:Molex_PicoBlade_53398-0371_1x03-1MP_P1.25mm_Vertical -> Connector_PinHeader_2.54mm:PinHeader_1x03_P2.54mm_Vertical
- R10: value 10k -> 15k
- R11: value 0R/R-Ipropi -> 10k
- R12: value 0R/R-Imode -> 52.3k
- R17: value 0R -> 10k
- R18: value 0R -> 0R/R-Ipropi
- R19: value 0R -> 0R/R-Imode
- R24: value 1000k -> 100k
- R25, R26: value 220R -> 15R
- R27: value 220R -> 0R
- R28: value 220R -> 1000k
- R29, R30: value 10k -> 220R
- R31: value 100R -> 220R
- U3: value 24CW1280T-I/OT -> AP62301Z6; footprint Package_TO_SOT_SMD:SOT-23-5 -> Package_TO_SOT_SMD:SOT-563
- U4: value ESP32-S3-WROOM-1 -> 24CW1280T-I/OT; footprint PCM_Espressif:ESP32-S3-WROOM-1 -> Package_TO_SOT_SMD:SOT-23-5
- U5: value USBLC6-2SC6 -> ESP32-S3-WROOM-1; footprint Package_TO_SOT_SMD:TSOT-23-6_HandSoldering -> PCM_Espressif:ESP32-S3-WROOM-1
- U6: value BMI088 -> USBLC6-2SC6; footprint finca:PQFN50P450X300X100-16N -> Package_TO_SOT_SMD:TSOT-23-6_HandSoldering
- moved D3 145.6 mm to (23.2, 65.9)
- moved D4 145.6 mm to (23.2, 68.9)
- moved D5 145.6 mm to (23.2, 72.0)
- moved D6 145.6 mm to (23.2, 75.0)
- moved D7 145.6 mm to (23.2, 78.0)
- moved C19 142.9 mm to (226.4, 60.4)
- moved C18 142.9 mm to (226.4, 57.4)
- moved R17 136.5 mm to (231.2, 57.4)
- moved R18 136.5 mm to (231.2, 60.4)
- moved R19 136.5 mm to (231.2, 63.3)
- moved R28 132.0 mm to (19.0, 65.8)
- moved IC3 128.0 mm to (222.4, 52.6)
- moved C10 122.1 mm to (34.2, 75.2)
- moved R29 118.1 mm to (19.0, 68.8)
- moved R9 117.5 mm to (37.8, 66.0)
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Connections:
- C12 pad 1: Net-(IC2-CPL) -> +12V
- C12 pad 2: Net-(IC2-CPH) -> GND
- C13 pad 1: Net-(IC2-VCP) -> Net-(U3-SW)
- C13 pad 2: +12V -> Net-(U3-BST)
- C14 pad 1: Net-(IC3-CPL) -> VOUT_5V
- C14 pad 2: Net-(IC3-CPH) -> GND
- C15 pad 1: Net-(IC3-VCP) -> VOUT_5V
- C15 pad 2: +12V -> GND
- C18 pad 1: +12V -> Net-(IC3-CPL)
- C18 pad 2: GND -> Net-(IC3-CPH)
- C19 pad 1: +12V -> Net-(IC3-VCP)
- C19 pad 2: GND -> +12V
- C21 pad 1: +3V3 -> GND
- C21 pad 2: GND -> +12V
- C23 pad 1: GND -> +12V
- C23 pad 2: /CONNECTIVITY/SHLD -> GND
- C24 pad 1: VBUS_USB -> +3V3
- C25 pad 1: EN -> +3V3
- C26 pad 1: BOOT -> +3V3
- C27 pad 1: +3V3 -> GND
- C27 pad 2: GND -> /CONNECTIVITY/SHLD
- C28 pad 1: GND -> VBUS_USB
- C28 pad 2: +3.3V -> GND
- C29 pad 1: +3V3 -> EN
- C30 pad 1: GND -> BOOT
- C30 pad 2: +3.3V -> GND
- R10 pad 1: +3V3 -> +12V
- R10 pad 2: nFAULT -> Net-(U3-EN)
- R11 pad 1: GND -> Net-(U3-EN)
- R11 pad 2: Net-(IC2-IPROPI) -> GND
- R12 pad 1: GND -> VOUT_5V
- R12 pad 2: Net-(IC2-IMODE) -> Net-(U3-FB)
- R13 pad 1: +3V3 -> Net-(U3-FB)
- R13 pad 2: nFAULT -> GND
- R17 pad 1: PMODE_2 -> nFAULT
- R18 pad 1: PMODE_1 -> GND
- R18 pad 2: GND -> Net-(IC3-IPROPI)
- R19 pad 1: PMODE_2 -> GND
- R19 pad 2: GND -> Net-(IC3-IMODE)
- R24 pad 1: Net-(D3-K) -> /CONNECTIVITY/SHLD
- R25 pad 1: Net-(D4-K) -> D_NEG_IN
- R25 pad 2: GND -> Net-(R25-Pad2)
- R26 pad 1: Net-(D5-K) -> D_POS_IN
- R26 pad 2: GND -> Net-(R26-Pad2)
- R27 pad 1: Net-(D6-K) -> BZ1_PWM
- R27 pad 2: GND -> Net-(BZ1-+)
- R28 pad 1: Net-(D7-K) -> Net-(D3-K)
- R29 pad 1: EN -> Net-(D4-K)
- R29 pad 2: +3V3 -> GND
- R30 pad 1: +3V3 -> Net-(D5-K)
- R30 pad 2: QRE_BACK -> GND
- R31 pad 1: +3V3 -> Net-(D6-K)
- R31 pad 2: Net-(J8-Pin_2) -> GND
- U3 pad 1: SCL -> GND
- U3 pad 2: GND -> Net-(U3-SW)
- U3 pad 3: SDA -> +12V
- U3 pad 4: +3V3 -> Net-(U3-FB)
- U3 pad 5: unconnected-(U3-WP-Pad5) -> Net-(U3-EN)
- U4 pad 1: GND -> SCL
- U4 pad 2: +3V3 -> GND
- U4 pad 3: EN -> SDA
- U4 pad 4: unconnected-(U4-IO4-Pad4) -> +3V3
- U5 pad 1: Net-(R21-Pad2) -> GND
- U5 pad 2: GND -> +3V3
- U5 pad 3: Net-(R22-Pad2) -> EN
- U5 pad 4: D- -> unconnected-(U5-IO4-Pad4)
- U5 pad 5: VBUS_USB -> unconnected-(U5-IO5-Pad5)
- U5 pad 6: D+ -> unconnected-(U5-IO6-Pad6)
- U6 pad 1: unconnected-(U6-INT2-Pad1) -> Net-(R25-Pad2)
- U6 pad 2: unconnected-(U6-NC-Pad2) -> GND
- U6 pad 3: +3.3V -> Net-(R26-Pad2)
- U6 pad 4: GND -> D+
- U6 pad 5: unconnected-(U6-CSB2-Pad5) -> VBUS_USB
- U6 pad 6: GND -> D-
Routing:
- net VBATT_SHUNT: track 0.00 -> 9.34 mm
- net Net-(R25-Pad2): track 0.00 -> 8.64 mm
- net Net-(IC2-VCP): track 0.00 -> 8.64 mm, vias 0 -> 2
- net +3V3: track 0.00 -> 8.16 mm, vias 0 -> 2
- net PMODE_1: track 0.00 -> 6.98 mm
- net D+: track 0.00 -> 6.53 mm
- net Net-(IC2-CPL): track 0.00 -> 5.53 mm
- net VBUS_USB: track 0.00 -> 5.42 mm, vias 0 -> 1
- net VBATT: track 0.00 -> 5.30 mm
- net +12V: track 0.00 -> 4.33 mm
- net D-: track 0.00 -> 4.05 mm
- net VOLTAGE_ALERT: track 0.00 -> 4.01 mm
- net MOTOR_R_1: track 0.00 -> 3.52 mm, vias 0 -> 2
- net EN_R: track 0.00 -> 3.52 mm, vias 0 -> 2
- net Net-(IC2-IMODE): track 0.00 -> 3.38 mm, vias 0 -> 2
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Other:
- board size 84.8 x 79.1 mm -> 97 x 30 mm
- board text added: "- DEAL WITH THIS"
- board text added: "5V CONV"
- board text added: "BACK"
- board text added: "FRONT"
- board text added: "LEDS"
- board text added: "LEFT"
- board text added: "MOTOR CONTROL"
- board text added: "RIGHT"

Commit message: minor schematic update
Parts:
- removed H2, H3: Mounting Hole M3, MountingHole:MountingHole_3.2mm_M3_Pad_Via
- C25, C26, R33: moved to F.Cu
- moved H1 7.50 mm to (86.0, 82.8)
- moved H4 7.50 mm to (175.5, 82.8)
- moved R33 5.16 mm to (91.0, 55.5), turned to -90 degrees
- moved C25 5.00 mm to (90.2, 51.6), turned to 180 degrees
- moved C26 1.09 mm to (93.0, 57.2)
Routing:
- net +3V3: track 8.16 -> 3.19 mm
Other:
- board size 97 x 30 mm -> 97 x 37.5 mm

Commit message: PCB update MKV
Parts:
- added H2: Mounting Hole M3, MountingHole:MountingHole_3.2mm_M3_Pad_Via, F.Cu at (60.6, 30.7)
- added H3: Mounting Hole M3, MountingHole:MountingHole_3.2mm_M3_Pad_Via, F.Cu at (68.6, 30.7)
- C25, D1, D2, R30, R31, R32, R33: moved to B.Cu
- J1, Q1, R5: moved to F.Cu
- moved R28 168.0 mm to (186.8, 74.8), turned to -90 degrees
- moved D3 163.6 mm to (186.8, 70.5), turned to 90 degrees
- moved R30 74.3 mm to (90.8, 52.5), turned to -90 degrees
- moved R31 72.2 mm to (87.8, 52.5), turned to -90 degrees
- moved R32 70.4 mm to (84.8, 52.5), turned to -90 degrees
- moved D5 70.3 mm to (90.8, 52.2), turned to -90 degrees
- moved R29 69.2 mm to (88.2, 71.2)
- moved D6 68.4 mm to (87.8, 52.2), turned to -90 degrees
- moved D7 66.7 mm to (84.8, 52.2), turned to -90 degrees
- moved D4 61.3 mm to (84.3, 73.2)
- moved C31 58.3 mm to (146.1, 66.5), turned to -90 degrees
- moved C16 53.3 mm to (193.9, 36.1)
- moved C20 53.3 mm to (190.1, 36.1)
- moved C22 53.3 mm to (191.9, 38.2)
- moved IC2 53.3 mm to (192.6, 31.2)
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Connections:
- D4 pad 1: Net-(D4-K) -> GND
- D4 pad 2: VBUS 5V -> Net-(D4-A)
- R29 pad 1: Net-(D4-K) -> VBUS_USB
- R29 pad 2: GND -> Net-(D4-A)
Routing:
- net VBUS_USB: track 5.42 -> 0.48 mm, vias 1 -> 0
- net Net-(IC2-VCP): track 8.64 -> 5.22 mm
- net +5V: track 3.35 -> 0.00 mm
- net VBATT: track 5.30 -> 2.71 mm
- net GND: track 0.00 -> 2.36 mm
- net +3V3: track 3.19 -> 5.44 mm
Other:
- outline, holes or cut-outs redrawn
- board text removed: "LEDS"

Commit message: minor pcb update
Parts:
- BZ1, C1, JP1, R27, R3, R34, R35, R4, U1: moved to B.Cu
- moved C33 43.1 mm to (121.2, 66.5), turned to 90 degrees
- moved BZ1 28.7 mm to (171.0, 58.8), turned to 0 degrees
- moved U7 23.1 mm to (150.5, 67.2)
- moved C32 23.1 mm to (150.5, 64.3)
- moved C34 23.1 mm to (150.5, 70.1)
- moved R34 18.1 mm to (129.5, 48.5)
- moved R35 13.8 mm to (129.5, 46.2)
- moved SW1 11.3 mm to (173.8, 70.8), turned to 45 degrees
- moved C1 6.79 mm to (188.6, 82.2), turned to -90 degrees
- moved R4 5.78 mm to (191.4, 80.5), turned to 180 degrees
- moved R3 4.64 mm to (188.6, 86.0), turned to -90 degrees
- moved J13 4.61 mm to (154.0, 57.2)
- moved U1 4.15 mm to (191.3, 84.7), turned to 90 degrees
- moved C24 3.40 mm to (155.4, 64.5)
- moved U4 3.40 mm to (155.5, 67.6)
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Routing:
- net VBATT_SHUNT: track 9.34 -> 2.82 mm
- net +3V3: track 5.44 -> 9.95 mm
- net VOLTAGE_ALERT: track 4.01 -> 0.00 mm
- net VBUS_INA226: track 2.30 -> 4.49 mm
- net VBATT: track 2.71 -> 4.16 mm

Commit message: PCB Updtae MK5
Parts:
- removed the C16 at (193.9, 36.1)
- removed the C17 at (192.8, 36.0)
- removed the C20 at (190.1, 36.1)
- removed the C22 at (191.9, 38.2)
- removed H2, H3: Mounting Hole M3, MountingHole:MountingHole_3.2mm_M3_Pad_Via
- removed the IC2 at (192.6, 31.2)
- removed the JP2 at (196.7, 32.0)
- removed the R15 at (192.6, 29.1)
- removed the R16 at (190.7, 29.1)
- C19, R18, R19: moved to B.Cu
- R34, R35: moved to F.Cu
- moved R3 26.3 mm to (163.7, 77.6), turned to -135 degrees
- moved JP1 25.9 mm to (168.8, 80.8), turned to 45 degrees
- moved U1 25.5 mm to (166.6, 78.7), turned to 45 degrees
- moved R19 25.0 mm to (207.9, 54.2), turned to 90 degrees
- moved C1 23.4 mm to (166.3, 75.0), turned to -135 degrees
- moved R4 22.4 mm to (169.6, 75.8), turned to 135 degrees
- moved R18 22.2 mm to (209.8, 54.2), turned to 90 degrees
- moved D3 20.8 mm to (170.6, 57.5)
- moved R28 20.8 mm to (170.5, 61.8)
- moved C21 19.3 mm to (207.2, 61.2)
- moved JP3 17.5 mm to (213.9, 57.1), turned to 90 degrees
- moved Q2 17.4 mm to (176.9, 64.6), turned to 45 degrees
- moved C19 16.4 mm to (210.0, 61.1), turned to 180 degrees
- moved C18 15.8 mm to (211.1, 61.2), turned to 180 degrees
- moved R17 15.2 mm to (216.5, 53.5), turned to -90 degrees
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Routing:
- net VBATT_SHUNT: track 2.82 -> 12.2 mm, vias 0 -> 2
- net GND: track 2.36 -> 7.02 mm
- net Net-(IC2-VCP): track 5.22 -> 0.90 mm, vias 2 -> 1
- net PMODE_1: track 6.98 -> 3.49 mm
- net Net-(IC2-CPL): track 5.53 -> 2.77 mm
- net +12V: track 4.33 -> 2.16 mm
- net MOTOR_R_1: track 3.52 -> 1.76 mm, vias 2 -> 1
- net EN_R: track 3.52 -> 1.76 mm, vias 2 -> 1
- net MOTOR_L_1: track 0.00 -> 1.76 mm, vias 0 -> 1
- net EN_L: track 0.00 -> 1.76 mm, vias 0 -> 1
- net Net-(Q2-G): track 0.00 -> 1.69 mm
- net Net-(IC2-IMODE): track 3.38 -> 1.69 mm, vias 2 -> 1
- net PH_R: track 3.35 -> 1.68 mm, vias 2 -> 1
- net PH_L: track 0.00 -> 1.68 mm, vias 0 -> 1
- net Net-(IC3-IMODE): track 0.00 -> 1.66 mm, vias 0 -> 1
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- added copper zone on B.Cu, net VBATT
Other:
- board text removed: "MOTOR CONTROL"

Commit message: PCB and 3d update
Parts:
- moved C18 51.4 mm to (160.3, 68.9)
- moved C19 51.4 mm to (159.2, 68.8)
- moved C21 51.4 mm to (156.5, 68.9)
- moved C23 51.4 mm to (158.2, 71.0)
- moved IC3 51.4 mm to (158.9, 64.0)
- moved JP3 51.4 mm to (163.1, 64.8)
- moved R17 51.4 mm to (165.7, 61.2)
- moved R18 51.4 mm to (159.0, 61.9)
- moved R19 51.4 mm to (157.1, 61.9)
- moved C24 44.0 mm to (115.6, 83.2)
- moved C32 44.0 mm to (110.7, 83.2)
- moved C34 44.0 mm to (110.7, 88.7)
- moved U4 44.0 mm to (115.7, 86.3)
- moved U7 44.0 mm to (110.7, 86.0)
- moved J13 7.45 mm to (161.5, 57.0)
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