File: main_hw/SUMEC_MK_V/SUMEC_MK_V.kicad_pcb (KiCad board)
At the start: 4 copper layers, 97 x 37.5 mm, 119 parts, among them IC1 TPS565242DRLR, IC2 DRV8874PWPR, IC3 DRV8874PWPR, J1 XT30PW-M, J10 Conn_01x03_Pin, J11 Conn_01x03_Pin, J12 Conn_01x03_Pin, J13 Conn_01x03_Pin, J14 Conn_01x03_Pin, J15 Conn_01x03_Pin, J2 Conn_01x06_Socket, J3 Conn_01x06_Socket, J4 USB_TypeC, J5 Conn_01x04_Pin, J6 Conn_01x06_Pin, J7 Conn_01x06_Pin, J8 Conn_01x03_Pin, J9 Conn_01x06_Pin, Q1 Q_PMOS, Q2 Q_PMOS, SW1 SW_DPDT_x2, SW2 SW_Push, SW3 SW_Push, SW4 SW_Push, SW5 SW_Push, U1 INA226, U2 TPS62133, U3 AP62301Z6, U4 24CW1280T-I/OT, U5 ESP32-S3-WROOM-1, U6 USBLC6-2SC6, U7 BMI088

Commit message: pcb update
Parts:
- R28: value 1000k -> 1k
- moved SW1 85.9 mm to (87.8, 72.0), turned to 135 degrees
- moved R6 81.1 mm to (84.5, 70.5), turned to 135 degrees
- moved Q2 76.8 mm to (86.8, 68.3), turned to 45 degrees
- moved R4 76.8 mm to (93.5, 74.8), turned to -135 degrees
- moved C1 74.4 mm to (92.0, 78.7), turned to -45 degrees
- moved JP1 71.1 mm to (97.8, 76.3), turned to 135 degrees
- moved U1 70.9 mm to (95.7, 78.5), turned to 135 degrees
- moved R3 69.2 mm to (94.6, 81.4), turned to -45 degrees
- moved C32 69.0 mm to (96.9, 93.2)
- moved C34 69.0 mm to (91.4, 93.2)
- moved U7 69.0 mm to (94.2, 93.2)
- moved C24 69.0 mm to (94.6, 101.6)
- moved U4 69.0 mm to (94.6, 98.8)
- moved J1 66.6 mm to (97.7, 80.8), turned to -135 degrees
- moved C12 47.7 mm to (168.0, 97.3)
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Connections:
- D5 pad 1: Net-(D5-K) -> GND
- D5 pad 2: LED_1 -> Net-(D5-A)
- D6 pad 1: Net-(D6-K) -> GND
- D6 pad 2: LED_2 -> Net-(D6-A)
- D7 pad 1: Net-(D7-K) -> GND
- D7 pad 2: LED_3 -> Net-(D7-A)
- R30 pad 1: Net-(D5-K) -> LED_1
- R30 pad 2: GND -> Net-(D5-A)
- R31 pad 1: Net-(D6-K) -> LED_2
- R31 pad 2: GND -> Net-(D6-A)
- R32 pad 1: Net-(D7-K) -> LED_3
- R32 pad 2: GND -> Net-(D7-A)
Routing:
- net +5V: track 92.4 -> 0.00 mm, vias 2 -> 1
- net VOUT_5V: track 78.0 -> 0.00 mm
- net +3V3: track 69.3 -> 1.00 mm, vias 18 -> 16
- net IR_MODULE: track 53.5 -> 0.00 mm
- net GND: track 36.1 -> 0.00 mm, vias 17 -> 16
- net BOOT: track 29.3 -> 0.00 mm
- net nSLEEP: track 28.5 -> 0.00 mm
- net nFAULT: track 28.3 -> 0.00 mm
- net PH_L: track 26.6 -> 0.00 mm
- net EN_L: track 26.2 -> 0.00 mm
- net EN: track 25.9 -> 0.00 mm
- net EN_R: track 25.0 -> 0.00 mm
- net PH_R: track 24.8 -> 0.00 mm
- net QRE_BACK: track 16.7 -> 0.00 mm
- net VBUS_USB: track 16.3 -> 0.00 mm, vias 1 -> 0
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- removed copper zone on In2.Cu, net +3V3
- removed copper zone on B.Cu, net /POWER_SUPPLY/FET_SW
- removed copper zone on F.Cu, net /POWER_SUPPLY/FET_SW
- removed copper zone on F.Cu, net VBATT_SHUNT
Other:
- outline, holes or cut-outs redrawn
- board text removed: "EEPROwoM"
- board text removed: "LEDS"

Commit message: PCB routing update
Parts:
- C12, C13, C14, C15, JP2, JP3, L3, Q2, R10, R11, R12, R13, R29, R5, R6, U3: moved to B.Cu
- moved D3 94.2 mm to (104.5, 70.0)
- moved R28 94.2 mm to (104.5, 70.2)
- moved C23 82.1 mm to (107.3, 67.8), turned to -90 degrees
- moved C18 80.0 mm to (109.4, 69.8), turned to 90 degrees
- moved C14 78.8 mm to (105.2, 54.3)
- moved C22 77.2 mm to (107.2, 58.9), turned to -90 degrees
- moved C21 76.9 mm to (109.4, 66.0), turned to -90 degrees
- moved L3 76.9 mm to (100.2, 55.9)
- moved C15 75.6 mm to (106.3, 57.1), turned to -90 degrees
- moved C12 75.0 mm to (104.3, 57.7), turned to 90 degrees
- moved C19 74.7 mm to (113.5, 67.5), turned to 90 degrees
- moved C16 73.9 mm to (109.3, 61.0), turned to 90 degrees
- moved U3 73.4 mm to (102.0, 59.2)
- moved C13 73.3 mm to (98.7, 59.3)
- moved JP3 73.1 mm to (115.2, 70.8)
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Connections:
- D3 pad 1: Net-(D3-K) -> GND
- D3 pad 2: +12V -> Net-(D3-A)
- R28 pad 1: Net-(D3-K) -> +12V
- R28 pad 2: GND -> Net-(D3-A)
Routing:
- net +12V: track 0.00 -> 9.82 mm
- net +5V: track 0.00 -> 4.93 mm
- net unconnected-(U5-IO42-Pad35): vias 1 -> 0
- net unconnected-(U5-IO40-Pad33): vias 2 -> 0
- net VBATT_SHUNT: vias 3 -> 5
- net SHARP_R: vias 0 -> 2
- net Net-(IC3-IPROPI): vias 1 -> 0
- net MOTOR_L_1: vias 1 -> 0
- net +3V3: vias 16 -> 14
- added copper zone on B.Cu, net +12V
- added copper zone on B.Cu, net /POWER_SUPPLY/FET_SW
- added copper zone on B.Cu, net /POWER_SUPPLY/SW
- added copper zone on B.Cu, net FB
- added copper zone on B.Cu, net VBATT_SHUNT
- added copper zone on F.Cu, net VBATT_SHUNT
- removed copper zone on F.Cu, net /POWER_SUPPLY/SW
- removed copper zone on F.Cu, net FB

Commit message: a lot of routing and layout updates
Parts:
- removed C10: 22uF, Capacitor_Tantalum_SMD:CP_EIA-2012-12_Kemet-R_Pad1.30x1.05mm_HandSolder
- removed C2: 3.3nF, Capacitor_SMD:C_0805_2012Metric_Pad1.18x1.45mm_HandSolder
- removed C4: 10uF, Capacitor_Tantalum_SMD:CP_EIA-3216-18_Kemet-A_Pad1.58x1.35mm_HandSolder
- removed C6: 100nF, Capacitor_SMD:C_0805_2012Metric_Pad1.18x1.45mm_HandSolder
- removed J7, J9: Conn_01x06_Pin, Connector_Molex:Molex_PicoBlade_53398-0671_1x06-1MP_P1.25mm_Vertical
- removed L2: 2.2uH, Inductor_SMD:L_Vishay_IHLP-1616
- removed R9: 100k, Resistor_SMD:R_0805_2012Metric_Pad1.20x1.40mm_HandSolder
- removed U2: TPS62133, Package_DFN_QFN:VQFN-16-1EP_3x3mm_P0.5mm_EP1.68x1.68mm_ThermalVias
- BZ1, C33, R27: moved to F.Cu
- moved R37 41.7 mm to (139.2, 63.4), turned to 180 degrees
- moved R36 41.4 mm to (139.2, 61.5), turned to 180 degrees
- moved C24 39.4 mm to (117.0, 75.8)
- moved U4 39.4 mm to (114.2, 75.8)
- moved C9 25.7 mm to (145.2, 65.3), turned to 90 degrees
- moved TP9 24.3 mm to (178.0, 57.5), turned to 180 degrees
- moved C7 23.7 mm to (147.0, 65.3), turned to 90 degrees
- moved C8 21.8 mm to (148.8, 65.3), turned to 90 degrees
- moved R8 21.4 mm to (145.9, 70.2), turned to 180 degrees
- moved TP7 21.0 mm to (178.0, 63.5), turned to 180 degrees
- moved R7 20.8 mm to (147.4, 68.2), turned to 0 degrees
- moved TP10 20.7 mm to (178.0, 54.5), turned to 180 degrees
- moved TP8 20.2 mm to (178.0, 60.5), turned to 180 degrees
- moved C11 20.0 mm to (150.7, 65.3), turned to 90 degrees
- moved SW4 19.2 mm to (87.8, 52.2)
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Connections:
- net /POWER_SUPPLY/FB_5V renamed /POWER/FB_5V
- net /POWER_SUPPLY/FET_SW renamed /POWER/FET_SW
- net /POWER_SUPPLY/SW renamed /POWER/SW
- SW3 pad 1: +3V3 -> GND
- SW3 pad 2: BUTTON_IO_48 -> BTN_IOXX
- SW4 pad 1: +3V3 -> GND
- SW4 pad 2: BUTTON_IO_47 -> BTN_IOXY
- TP11 pad 1: IR MODULE -> IR_MODULE
- U5 pad 10: unconnected-(U5-IO17-Pad10) -> nSLEEP
- U5 pad 11: unconnected-(U5-IO18-Pad11) -> PH_L
- U5 pad 12: unconnected-(U5-IO8-Pad12) -> EN_L
- U5 pad 17: unconnected-(U5-IO9-Pad17) -> VOLTAGE_ALERT
- U5 pad 18: unconnected-(U5-IO10-Pad18) -> SHARP_L
- U5 pad 19: unconnected-(U5-IO11-Pad19) -> POL_M
- U5 pad 20: unconnected-(U5-IO12-Pad20) -> POL_R
- U5 pad 21: unconnected-(U5-IO13-Pad21) -> QRE_R
- U5 pad 22: unconnected-(U5-IO14-Pad22) -> QRE_L
- U5 pad 31: unconnected-(U5-IO38-Pad31) -> SHARP_R
- U5 pad 32: unconnected-(U5-IO39-Pad32) -> ACC_INT
- U5 pad 33: unconnected-(U5-IO40-Pad33) -> GYR_INT
- U5 pad 34: unconnected-(U5-IO41-Pad34) -> IR_MODULE
- U5 pad 35: unconnected-(U5-IO42-Pad35) -> SCL
- U5 pad 36: unconnected-(U5-IO44-Pad36) -> SDA
- U5 pad 37: unconnected-(U5-IO47-Pad37) -> LED_1
- U5 pad 38: unconnected-(U5-IO2-Pad38) -> LED_2
- U5 pad 39: unconnected-(U5-IO1-Pad39) -> LED_3
- U5 pad 4: unconnected-(U5-IO4-Pad4) -> BTN_IOXX
- U5 pad 5: unconnected-(U5-IO5-Pad5) -> BTN_IOXY
- U5 pad 6: unconnected-(U5-IO6-Pad6) -> PH_R
- U5 pad 7: unconnected-(U5-IO7-Pad7) -> EN_R
- U5 pad 8: unconnected-(U5-IO15-Pad8) -> nFAULT
- U5 pad 9: unconnected-(U5-IO16-Pad9) -> QRE_BACK
Routing:
- net +5V: track 4.93 -> 100.4 mm, vias 1 -> 5
- net SCL: track 0.00 -> 79.2 mm, vias 0 -> 5
- net SDA: track 0.00 -> 76.2 mm, vias 0 -> 5
- net IR_MODULE: track 0.00 -> 43.6 mm, vias 0 -> 2
- net VOLTAGE_ALERT: track 0.00 -> 41.1 mm, vias 0 -> 2
- net SHARP_L: track 0.00 -> 40.1 mm, vias 0 -> 2
- net BTN_IOXY: track 0.00 -> 38.4 mm, vias 0 -> 2
- net BOOT: track 0.00 -> 38.0 mm, vias 1 -> 2
- net VOUT_5V: track 0.00 -> 35.4 mm, vias 0 -> 1
- net D+: track 0.00 -> 32.8 mm
- net D-: track 0.00 -> 31.2 mm
- net MOTOR_R_2: track 0.00 -> 29.1 mm, vias 0 -> 2
- net BTN_IOXX: track 0.00 -> 28.5 mm, vias 0 -> 2
- net MOTOR_R_1: track 0.00 -> 25.0 mm, vias 1 -> 2
- net VBUS_USB: track 0.00 -> 24.7 mm, vias 0 -> 4
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- added copper zone on In2.Cu, net +12V
- added copper zone on In2.Cu, net +3V3
- added copper zone on B.Cu, net VOUT_5V
Other:
- board text added: "0"
- board text added: "0 mm"
- board text added: "0.01 mm"
- board text added: "0.02"
- board text added: "0.035 mm"
- board text added: "0.1 mm"
- board text added: "1"
- board text added: "1.24 mm"
- board text added: "3.3"
- board text added: "4.5"
- board text added: "B.Paste"
- board text added: "B.Silkscreen"
- board text added: "B.SolderMask"
- board text added: "Back.Cu"
- board text added: "Bottom Silk Screen"
- board text added: "Bottom Solder Mask"
- board text added: "Bottom Solder Paste"
- board text added: "Color"
- board text added: "Dielectric"
- board text added: "Epsilon R"
- board text added: "F.Paste"
- board text added: "F.Silkscreen"
- board text added: "F.SolderMask"
- board text added: "FR4"
- board text added: "FR4 natural"
- board text added: "Front.Cu"
- board text added: "In1.Cu"
- board text added: "In2.Cu"
- board text added: "Layer Name"
- board text added: "Loss Tangent"
- board text added: "Material"
- board text added: "Not specified"
- board text added: "Thickness (mm)"
- board text added: "Top Silk Screen"
- board text added: "Top Solder Mask"
- board text added: "Top Solder Paste"
- board text added: "Type"
- board text added: "copper"
- board text added: "core"
- board text added: "prepreg"
- board text removed: "OLD 5V CONV"

Commit message: routing update
Parts:
- moved C26 1.17 mm to (120.8, 57.0), turned to 90 degrees
- moved C18 0.06 mm to (109.7, 69.8)
Routing:
- net +3V3: track 19.7 -> 85.4 mm, vias 11 -> 20
- net GND: track 10.0 -> 28.4 mm, vias 12 -> 21
- net FB: track 0.00 -> 4.12 mm
- net +5V: track 100.4 -> 102.1 mm, vias 5 -> 6
- net SHARP_R: track 11.7 -> 13.0 mm
- net IR_MODULE: track 43.6 -> 44.2 mm
