File: main_hw/SUMEC_MK_V/MOTOR_CONTROL.kicad_sch (KiCad schematic)
At the start: 20 parts, among them IC2 DRV8874PWPR, IC3 DRV8874PWPR

Commit message: MK V Schematic update
Parts:
- gave numbers to parts that had none: 4
Connections:
- net MOTOR_L_1: now also J14.6 (Pin_6); no longer J14.5 (Pin_5)
- net MOTOR_L_2: now also J14.5 (Pin_5); no longer J14.6 (Pin_6)
- net MOTOR_R_1: now also J12.6 (Pin_6); no longer J12.5 (Pin_5)
- net MOTOR_R_2: now also J12.5 (Pin_5); no longer J12.6 (Pin_6)
- net OUT 1A renamed OUT_R_A
- net OUT 1B renamed OUT_R_B
- net OUT 2A renamed OUT_L_A
- net OUT 2B renamed OUT_L_B
Other:
- note added: "MOTOR - LEFT"
- note added: "MOTOR - RIGHT"
- note removed: "M1"
- note removed: "M2"
- moved on the sheet: C11, C12, C13, C14, C15, C16, C17, C18, IC2, IC3, J12, J14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

Commit message: Schematic update - finalized
Parts:
- removed JP1, JP2: Solder Jumper, symbol Jumper:SolderJumper_3_Open
- added R16, R17, R18, R19: 0R, Resistor_SMD:R_0805_2012Metric_Pad1.20x1.40mm_HandSolder, symbol Device:R
- renumbered C11 to C12, C12 to C13, C13 to C14, C14 to C15, C15 to C16, C16 to C17, C17 to C18, C18 to C19, J12 to J2, J14 to J3, R8 to R10, R10 to R11, R6 to R12, R9 to R13, R11 to R14, R7 to R15
Connections:
- net +3V3: now also R16.2, R17.2
- net GND: now also R18.2, R19.2
- net PMODE_1: now also R16.1, R18.1
- net PMODE_2: now also R17.1, R19.1
Other:
- title: SUMEC_MK_IV -> SUMEC_MK_V

Commit message: MK V Schematic update
Parts:
- removed R10: 10k, Resistor_SMD:R_0805_2012Metric_Pad1.20x1.40mm_HandSolder, symbol Device:R_Small
- removed R16, R17, R18, R19: 0R, Resistor_SMD:R_0805_2012Metric_Pad1.20x1.40mm_HandSolder, symbol Device:R
- added JP2, JP3: SolderJumper_3_Open, Jumper:SolderJumper-3_P2.0mm_Open_TrianglePad1.0x1.5mm, symbol Jumper:SolderJumper_3_Open
- renumbered C12 to C16, C13 to C17, C14 to C18, C15 to C19, C16 to C20, C17 to C21, C18 to C22, C19 to C23, R11 to R15, R12 to R16, R13 to R17, R14 to R18, R15 to R19
Connections:
- net +3V3: now also R17.2, JP2.1 (A), JP3.1 (A); no longer R17.1
- net GND: now also JP2.3 (B), JP3.3 (B)
- net PMODE_1: now also JP2.2 (C)
- net PMODE_2: now also JP3.2 (C)
- net nFAULT: now also R17.1; no longer R17.2
Other:
- moved on the sheet: R17
