File: main_hw/SUMEC_MK_V/MECHANICS.kicad_sch (KiCad schematic)
At the start: 16 parts, among them SW2 SW_Push, SW3 SW_Push, SW4 SW_Push, SW5 SW_Push

Commit message: MK V Schematic update
Other:
- note added: "EN=reset, BOOT=bootloader mode Enable (EN) is the 3.3V regulator's enable pin. It's pulled up, so connect to ground to disable the 3.3V regulator. This means that you can use this pin connected to a pushbutton to restart your ESP32, for example."
- note added: "ENABLE RESET"
- note removed: "EN=RESET, BOOT=bootloader mode Enable (EN) is the 3.3V regulator's enable pin. It's pulled up, so connect to ground to disable the 3.3V regulator. This means that you can use this pin connected to a pushbutton to restart your ESP32, for example."
- note removed: "ENABLE"
- moved on the sheet: C23, C24, R15, SW2, SW3, SW4, SW5, TP1, TP2, TP3, TP4, TP5

Commit message: Schematic update - finalized
Parts:
- renumbered C23 to C25, C24 to C26, R15 to R29, TP4 to TP10, TP5 to TP11, TP1 to TP7, TP2 to TP8, TP3 to TP9
Other:
- title: SUMEC_MK_IV -> SUMEC_MK_V
Changed lines of the file:
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@@
 	(paper "A4")
 	(title_block
-		(title "SUMEC_MK_IV")
+		(title "SUMEC_MK_V")
 		(date "2024-08-05")
-		(rev "v3.0.9")
+		(rev "v.1.0.0")
 		(company "SPS NA PROSEKU")
 		(comment 1 "Made in Prague, Czech Republic")
 		(comment 2 "CONTACT: Savva Popov, savva.popov.sp@gmail.com, +420 605 570 366")
 		(comment 3 "Made by bismarx-v1")
-		(comment 4 "SUMEC MK IV aka SMD-V3 board")
+		(comment 4 "SUMEC MK V aka SMD-V4 board")
 	)
 	(rectangle
@@
 		(on_board yes)
 		(dnp no)
-		(property "Reference" "TP3"
+		(property "Reference" "TP9"
 			(at 147.828 48.768 0)
 			(effects
@@
 			(project "SUMEC_MK_V"
 				(path "/900bd7ac-cdf9-4a2f-8b1f-2c21e3760046/a907f0f2-2950-481d-8037-7b9f13f2e9c5"
-					(reference "TP3")
+					(reference "TP9")
 					(unit 1)
 				)
@@
 		(on_board yes)
 		(dnp no)
-		(property "Reference" "#PWR083"
+		(property "Reference" "#PWR071"
 			(at 133.35 53.34 0)
 			(effects
@@
 			(project "SUMEC_MK_V"
 				(path "/900bd7ac-cdf9-4a2f-8b1f-2c21e3760046/a907f0f2-2950-481d-8037-7b9f13f2e9c5"
-					(reference "#PWR083")
+					(reference "#PWR071")
 					(unit 1)
 				)
@@
 		(on_board yes)
 		(dnp no)
-		(property "Reference" "R15"
+		(property "Reference" "R29"
 			(at 114.935 95.25 0)
 			(effects
@@
 			(project "SUMEC_MK_V"
 				(path "/900bd7ac-cdf9-4a2f-8b1f-2c21e3760046/a907f0f2-2950-481d-8037-7b9f13f2e9c5"
-					(reference "R15")
+					(reference "R29")
 					(unit 1)
 				)
@@
 		(on_board yes)
 		(dnp no)
-		(property "Reference" "#PWR048"
+		(property "Reference" "#PWR070"
 			(at 130.81 118.11 0)
 			(effects
@@
 			(project "SUMEC_MK_V"
 				(path "/900bd7ac-cdf9-4a2f-8b1f-2c21e3760046/a907f0f2-2950-481d-8037-7b9f13f2e9c5"
-					(reference "#PWR048")
+					(reference "#PWR070")
 					(unit 1)
 				)
@@
 		(on_board yes)
 		(dnp no)
-		(property "Reference" "#PWR047"
+		(property "Reference" "#PWR069"
 			(at 127 125.73 0)
 			(effects
@@
 			(project "SUMEC_MK_V"
 				(path "/900bd7ac-cdf9-4a2f-8b1f-2c21e3760046/a907f0f2-2950-481d-8037-7b9f13f2e9c5"
-					(reference "#PWR047")
+					(reference "#PWR069")
 					(unit 1)
 				)
@@
 		(on_board yes)
 		(dnp no)
-		(property "Reference" "C23"
+		(property "Reference" "C25"
 			(at 122.555 110.49 90)
 			(effects
@@
 			(project "SUMEC_MK_V"
 				(path "/900bd7ac-cdf9-4a2f-8b1f-2c21e3760046/a907f0f2-2950-481d-8037-7b9f13f2e9c5"
-					(reference "C23")
+					(reference "C25")
 					(unit 1)
 				)
@@
 		(on_board yes)
 		(dnp no)
-		(property "Reference" "TP5"
+		(property "Reference" "TP11"
 			(at 173.228 48.768 0)
 			(effects
@@
 			(project "SUMEC_MK_V"
 				(path "/900bd7ac-cdf9-4a2f-8b1f-2c21e3760046/a907f0f2-2950-481d-8037-7b9f13f2e9c5"
-					(reference "TP5")
+					(reference "TP11")
 					(unit 1)
 				)
@@
 		(on_board yes)
 		(dnp no)
-		(property "Reference" "C24"
+		(property "Reference" "C26"
 			(at 149.225 110.49 90)
 			(effects
@@
 			(project "SUMEC_MK_V"
 				(path "/900bd7ac-cdf9-4a2f-8b1f-2c21e3760046/a907f0f2-2950-481d-8037-7b9f13f2e9c5"
-					(reference "C24")
+					(reference "C26")
 					(unit 1)
 				)
@@
 		(at 58.42 62.23 90)
 		(unit 1)
-		(exclude_from_sim yes)
+		(exclude_from_sim no)
 		(in_bom no)
 		(on_board yes)
@@
 		(on_board yes)
 		(dnp no)
-		(property "Reference" "TP4"
+		(property "Reference" "TP10"
 			(at 160.528 48.768 0)
 			(effects
@@
 			(project "SUMEC_MK_V"
 				(path "/900bd7ac-cdf9-4a2f-8b1f-2c21e3760046/a907f0f2-2950-481d-8037-7b9f13f2e9c5"
-					(reference "TP4")
+					(reference "TP10")
 					(unit 1)
 				)
@@
 		(at 58.42 55.88 90)
 		(unit 1)
-		(exclude_from_sim yes)
+		(exclude_from_sim no)
 		(in_bom no)
 		(on_board yes)
@@
 		(on_board yes)
 		(dnp no)
-		(property "Reference" "TP2"
+		(property "Reference" "TP8"
 			(at 135.128 48.768 0)
 			(effects
@@
 			(project "SUMEC_MK_V"
 				(path "/900bd7ac-cdf9-4a2f-8b1f-2c21e3760046/a907f0f2-2950-481d-8037-7b9f13f2e9c5"
-					(reference "TP2")
+					(reference "TP8")
 					(unit 1)
 				)
@@
 		(on_board yes)
 		(dnp no)
-		(property "Reference" "#PWR045"
+		(property "Reference" "#PWR067"
 			(at 118.11 95.25 0)
 			(effects
@@
 			(project "SUMEC_MK_V"
 				(path "/900bd7ac-cdf9-4a2f-8b1f-2c21e3760046/a907f0f2-2950-481d-8037-7b9f13f2e9c5"
-					(reference "#PWR045")
+					(reference "#PWR067")
 					(unit 1)
 				)
@@
 		(on_board yes)
 		(dnp no)
-		(property "Reference" "#PWR081"
+		(property "Reference" "#PWR066"
 			(at 74.93 69.85 0)
 			(effects
@@
 			(project "SUMEC_MK_V"
 				(path "/900bd7ac-cdf9-4a2f-8b1f-2c21e3760046/a907f0f2-2950-481d-8037-7b9f13f2e9c5"
-					(reference "#PWR081")
+					(reference "#PWR066")
 					(unit 1)
 				)
@@
 		(at 58.42 49.53 90)
 		(unit 1)
-		(exclude_from_sim yes)
+		(exclude_from_sim no)
 		(in_bom no)
 		(on_board yes)
@@
 		(at 58.42 43.18 90)
 		(unit 1)
-		(exclude_from_sim yes)
+		(exclude_from_sim no)
 		(in_bom no)
 		(on_board yes)
@@
 		(on_board yes)
 		(dnp no)
-		(property "Reference" "TP1"
+		(property "Reference" "TP7"
 			(at 122.428 48.768 0)
 			(effects
@@
 			(project "SUMEC_MK_V"
 				(path "/900bd7ac-cdf9-4a2f-8b1f-2c21e3760046/a907f0f2-2950-481d-8037-7b9f13f2e9c5"
-					(reference "TP1")
+					(reference "TP7")
 					(unit 1)
 				)
@@
 		(on_board yes)
 		(dnp no)
-		(property "Reference" "#PWR049"
+		(property "Reference" "#PWR072"
 			(at 140.97 118.11 0)
 			(effects
@@
 			(project "SUMEC_MK_V"
 				(path "/900bd7ac-cdf9-4a2f-8b1f-2c21e3760046/a907f0f2-2950-481d-8037-7b9f13f2e9c5"
-					(reference "#PWR049")
+					(reference "#PWR072")
 					(unit 1)
 				)
@@
 		(on_board yes)
 		(dnp no)
-		(property "Reference" "#PWR082"
+		(property "Reference" "#PWR068"
 			(at 120.65 53.34 0)
 			(effects
@@
 			(project "SUMEC_MK_V"
 				(path "/900bd7ac-cdf9-4a2f-8b1f-2c21e3760046/a907f0f2-2950-481d-8037-7b9f13f2e9c5"
-					(reference "#PWR082")
+					(reference "#PWR068")
 					(unit 1)
 				)

Commit message: MK V Schematic update
Parts:
- renumbered C25 to C29, C26 to C30, R29 to R33
Changed lines of the file:
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@@
 		(on_board yes)
 		(dnp no)
-		(property "Reference" "#PWR071"
+		(property "Reference" "#PWR078"
 			(at 133.35 53.34 0)
 			(effects
@@
 			(project "SUMEC_MK_V"
 				(path "/900bd7ac-cdf9-4a2f-8b1f-2c21e3760046/a907f0f2-2950-481d-8037-7b9f13f2e9c5"
-					(reference "#PWR071")
+					(reference "#PWR078")
 					(unit 1)
 				)
@@
 		(on_board yes)
 		(dnp no)
-		(property "Reference" "R29"
+		(property "Reference" "R33"
 			(at 114.935 95.25 0)
 			(effects
@@
 			(project "SUMEC_MK_V"
 				(path "/900bd7ac-cdf9-4a2f-8b1f-2c21e3760046/a907f0f2-2950-481d-8037-7b9f13f2e9c5"
-					(reference "R29")
+					(reference "R33")
 					(unit 1)
 				)
@@
 		(on_board yes)
 		(dnp no)
-		(property "Reference" "#PWR070"
+		(property "Reference" "#PWR077"
 			(at 130.81 118.11 0)
 			(effects
@@
 			(project "SUMEC_MK_V"
 				(path "/900bd7ac-cdf9-4a2f-8b1f-2c21e3760046/a907f0f2-2950-481d-8037-7b9f13f2e9c5"
-					(reference "#PWR070")
+					(reference "#PWR077")
 					(unit 1)
 				)
@@
 		(on_board yes)
 		(dnp no)
-		(property "Reference" "#PWR069"
+		(property "Reference" "#PWR076"
 			(at 127 125.73 0)
 			(effects
@@
 			(project "SUMEC_MK_V"
 				(path "/900bd7ac-cdf9-4a2f-8b1f-2c21e3760046/a907f0f2-2950-481d-8037-7b9f13f2e9c5"
-					(reference "#PWR069")
+					(reference "#PWR076")
 					(unit 1)
 				)
@@
 		(on_board yes)
 		(dnp no)
-		(property "Reference" "C25"
+		(property "Reference" "C29"
 			(at 122.555 110.49 90)
 			(effects
@@
 			(project "SUMEC_MK_V"
 				(path "/900bd7ac-cdf9-4a2f-8b1f-2c21e3760046/a907f0f2-2950-481d-8037-7b9f13f2e9c5"
-					(reference "C25")
+					(reference "C29")
 					(unit 1)
 				)
@@
 		(on_board yes)
 		(dnp no)
-		(property "Reference" "C26"
+		(property "Reference" "C30"
 			(at 149.225 110.49 90)
 			(effects
@@
 			(project "SUMEC_MK_V"
 				(path "/900bd7ac-cdf9-4a2f-8b1f-2c21e3760046/a907f0f2-2950-481d-8037-7b9f13f2e9c5"
-					(reference "C26")
+					(reference "C30")
 					(unit 1)
 				)
@@
 		(on_board yes)
 		(dnp no)
-		(property "Reference" "#PWR067"
+		(property "Reference" "#PWR074"
 			(at 118.11 95.25 0)
 			(effects
@@
 			(project "SUMEC_MK_V"
 				(path "/900bd7ac-cdf9-4a2f-8b1f-2c21e3760046/a907f0f2-2950-481d-8037-7b9f13f2e9c5"
-					(reference "#PWR067")
+					(reference "#PWR074")
 					(unit 1)
 				)
@@
 		(on_board yes)
 		(dnp no)
-		(property "Reference" "#PWR066"
+		(property "Reference" "#PWR073"
 			(at 74.93 69.85 0)
 			(effects
@@
 			(project "SUMEC_MK_V"
 				(path "/900bd7ac-cdf9-4a2f-8b1f-2c21e3760046/a907f0f2-2950-481d-8037-7b9f13f2e9c5"
-					(reference "#PWR066")
+					(reference "#PWR073")
 					(unit 1)
 				)
@@
 		(on_board yes)
 		(dnp no)
-		(property "Reference" "#PWR072"
+		(property "Reference" "#PWR079"
 			(at 140.97 118.11 0)
 			(effects
@@
 			(project "SUMEC_MK_V"
 				(path "/900bd7ac-cdf9-4a2f-8b1f-2c21e3760046/a907f0f2-2950-481d-8037-7b9f13f2e9c5"
-					(reference "#PWR072")
+					(reference "#PWR079")
 					(unit 1)
 				)
@@
 		(on_board yes)
 		(dnp no)
-		(property "Reference" "#PWR068"
+		(property "Reference" "#PWR075"
 			(at 120.65 53.34 0)
 			(effects
@@
 			(project "SUMEC_MK_V"
 				(path "/900bd7ac-cdf9-4a2f-8b1f-2c21e3760046/a907f0f2-2950-481d-8037-7b9f13f2e9c5"
-					(reference "#PWR068")
-					(unit 1)
-				)
+					(reference "#PWR075")
+					(unit 1)
+				)

Commit message: PCB Updtae MK5
Parts:
- removed H2, H3: Mounting Hole M3, MountingHole:MountingHole_3.2mm_M3_Pad_Via, symbol Mechanical:MountingHole_Pad
Other:
- moved on the sheet: H4
Changed lines of the file:
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@@
-	)
-	(junction
-		(at 74.93 62.23)
-		(diameter 0)
-		(color 0 0 0 0)
 	)
 	(junction
@@
 	)
 	(junction
-		(at 74.93 49.53)
-		(diameter 0)
-		(color 0 0 0 0)
-	)
-	(junction
-		(at 74.93 55.88)
+		(at 74.93 52.07)
 		(diameter 0)
 		(color 0 0 0 0)
@@
 	(wire
 		(pts
-			(xy 74.93 63.5) (xy 74.93 62.23)
+			(xy 74.93 52.07) (xy 74.93 58.42)
 		)
 		(stroke
@@
 	(wire
 		(pts
-			(xy 74.93 43.18) (xy 74.93 49.53)
-		)
-		(stroke
-			(width 0)
-			(type default)
-		)
-	)
-	(wire
-		(pts
-			(xy 60.96 55.88) (xy 74.93 55.88)
+			(xy 74.93 43.18) (xy 74.93 52.07)
 		)
 		(stroke
@@
 	(wire
 		(pts
-			(xy 74.93 55.88) (xy 74.93 62.23)
-		)
-		(stroke
-			(width 0)
-			(type default)
-		)
-	)
-	(wire
-		(pts
-			(xy 74.93 49.53) (xy 74.93 55.88)
-		)
-		(stroke
-			(width 0)
-			(type default)
-		)
-	)
-	(wire
-		(pts
 			(xy 124.46 125.73) (xy 124.46 133.35)
 		)
@@
 	(wire
 		(pts
-			(xy 60.96 49.53) (xy 74.93 49.53)
-		)
-		(stroke
-			(width 0)
-			(type default)
-		)
-	)
-	(wire
-		(pts
 			(xy 140.97 109.22) (xy 143.51 109.22)
 		)
@@
 	(wire
 		(pts
-			(xy 60.96 62.23) (xy 74.93 62.23)
+			(xy 60.96 52.07) (xy 74.93 52.07)
 		)
 		(stroke
@@
 	(symbol
 		(lib_id "Mechanical:MountingHole_Pad")
-		(at 58.42 62.23 90)
+		(at 58.42 52.07 90)
 		(unit 1)
 		(exclude_from_sim no)
@@
 		(dnp no)
 		(property "Reference" "H4"
-			(at 52.705 62.23 90)
+			(at 52.705 52.07 90)
 			(effects
 				(font
@@
 		)
 		(property "Value" "Mounting Hole M3"
-			(at 57.15 58.42 90)
+			(at 57.15 48.26 90)
 			(effects
 				(font
@@
 		)
 		(property "Footprint" "MountingHole:MountingHole_3.2mm_M3_Pad_Via"
-			(at 58.42 62.23 0)
+			(at 58.42 52.07 0)
 			(effects
 				(font
@@
 		)
 		(property "Datasheet" "~"
-			(at 58.42 62.23 0)
+			(at 58.42 52.07 0)
 			(effects
 				(font
@@
 		)
 		(property "Description" "Mounting Hole with connection"
-			(at 58.42 62.23 0)
+			(at 58.42 52.07 0)
 			(effects
 				(font
@@
 	)
 	(symbol
-		(lib_id "Mechanical:MountingHole_Pad")
-		(at 58.42 55.88 90)
-		(unit 1)
-		(exclude_from_sim no)
-		(in_bom no)
-		(on_board yes)
-		(dnp no)
-		(property "Reference" "H3"
-			(at 52.705 55.88 90)
-			(effects
-				(font
-					(size 1.27 1.27)
-				)
-			)
-		)
-		(property "Value" "Mounting Hole M3"
-			(at 57.15 52.07 90)
-			(effects
-				(font
-					(size 1.27 1.27)
-				)
-				(hide yes)
-			)
-		)
-		(property "Footprint" "MountingHole:MountingHole_3.2mm_M3_Pad_Via"
-			(at 58.42 55.88 0)
-			(effects
-				(font
-					(size 1.27 1.27)
-				)
-				(hide yes)
-			)
-		)
-		(property "Datasheet" "~"
-			(at 58.42 55.88 0)
-			(effects
-				(font
-					(size 1.27 1.27)
-				)
-				(hide yes)
-			)
-		)
-		(property "Description" "Mounting Hole with connection"
-			(at 58.42 55.88 0)
-			(effects
-				(font
-					(size 1.27 1.27)
-				)
-				(hide yes)
-			)
-		)
-		(pin "1"
-		)
-		(instances
-			(project "SUMEC_MK_V"
-				(path "/900bd7ac-cdf9-4a2f-8b1f-2c21e3760046/a907f0f2-2950-481d-8037-7b9f13f2e9c5"
-					(reference "H3")
-					(unit 1)
-				)
-			)
-		)
-	)
-	(symbol
 		(lib_id "Switch:SW_Push")
 		(at 132.08 125.73 0)
@@
 	(symbol
 		(lib_id "power:GND")
-		(at 74.93 63.5 0)
+		(at 74.93 58.42 0)
 		(unit 1)
 		(exclude_from_sim no)
@@
 		(dnp no)
 		(property "Reference" "#PWR073"
-			(at 74.93 69.85 0)
+			(at 74.93 64.77 0)
 			(effects
 				(font
@@
 		)
 		(property "Value" "GND"
-			(at 74.93 67.31 0)
+			(at 74.93 62.23 0)
 			(effects
 				(font
@@
 		)
 		(property "Footprint" ""
-			(at 74.93 63.5 0)
+			(at 74.93 58.42 0)
 			(effects
 				(font
@@
 		)
 		(property "Datasheet" ""
-			(at 74.93 63.5 0)
+			(at 74.93 58.42 0)
 			(effects
 				(font
@@
 		)
 		(property "Description" "Power symbol creates a global label with name \"GND\" , ground"
-			(at 74.93 63.5 0)
+			(at 74.93 58.42 0)
 			(effects
 				(font
@@
 					(unit 1)
 				)
-			)
-		)
-	)
-	(symbol
-		(lib_id "Mechanical:MountingHole_Pad")
-		(at 58.42 49.53 90)
-		(unit 1)
-		(exclude_from_sim no)
-		(in_bom no)
-		(on_board yes)
-		(dnp no)
-		(property "Reference" "H2"
-			(at 52.705 49.53 90)
-			(effects
-				(font
-					(size 1.27 1.27)
-				)
-			)
-		)
-		(property "Value" "Mounting Hole M3"
-			(at 57.15 45.72 90)
-			(effects
-				(font
-					(size 1.27 1.27)
-				)
-				(hide yes)
-			)
-		)
-		(property "Footprint" "MountingHole:MountingHole_3.2mm_M3_Pad_Via"
-			(at 58.42 49.53 0)
-			(effects
-				(font
-					(size 1.27 1.27)
-				)
-				(hide yes)
-			)
-		)
-		(property "Datasheet" "~"
-			(at 58.42 49.53 0)
-			(effects
-				(font
-					(size 1.27 1.27)
-				)
-				(hide yes)
-			)
-		)
-		(property "Description" "Mounting Hole with connection"
-			(at 58.42 49.53 0)
-			(effects
-				(font
-					(size 1.27 1.27)
-				)
-				(hide yes)
-			)
-		)
-		(pin "1"
-		)
-		(instances
-			(project "SUMEC_MK_V"
-				(path "/900bd7ac-cdf9-4a2f-8b1f-2c21e3760046/a907f0f2-2950-481d-8037-7b9f13f2e9c5"
-					(reference "H2")
-					(unit 1)
-				)

Commit message: a lot of routing and layout updates
Connections:
- net +3V3: no longer SW3.1, SW4.1
- net GND: now also SW3.1, SW4.1
- net BUTTON_IO_47 renamed BTN_IOXY
- net BUTTON_IO_48 renamed BTN_IOXX
- net IR MODULE renamed IR_MODULE
Other:
- moved on the sheet: H1, H4
Changed lines of the file:
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@@
 	)
 	(junction
-		(at 124.46 125.73)
+		(at 124.46 133.35)
 		(diameter 0)
 		(color 0 0 0 0)
@@
 	)
 	(junction
-		(at 74.93 52.07)
+		(at 74.93 54.61)
 		(diameter 0)
 		(color 0 0 0 0)
@@
 	(wire
 		(pts
-			(xy 74.93 52.07) (xy 74.93 58.42)
+			(xy 74.93 54.61) (xy 74.93 57.15)
 		)
 		(stroke
@@
 	(wire
 		(pts
-			(xy 74.93 43.18) (xy 74.93 52.07)
+			(xy 74.93 45.72) (xy 74.93 54.61)
+		)
+		(stroke
+			(width 0)
+			(type default)
+		)
+	)
+	(wire
+		(pts
+			(xy 124.46 134.62) (xy 124.46 133.35)
 		)
 		(stroke
@@
 	(wire
 		(pts
-			(xy 123.19 125.73) (xy 124.46 125.73)
-		)
-		(stroke
-			(width 0)
-			(type default)
-		)
-	)
-	(wire
-		(pts
 			(xy 140.97 102.87) (xy 142.24 102.87)
 		)
@@
 	(wire
 		(pts
-			(xy 60.96 43.18) (xy 74.93 43.18)
+			(xy 60.96 45.72) (xy 74.93 45.72)
 		)
 		(stroke
@@
 	(wire
 		(pts
-			(xy 60.96 52.07) (xy 74.93 52.07)
+			(xy 60.96 54.61) (xy 74.93 54.61)
 		)
 		(stroke
@@
 		)
 	)
-	(global_label "BUTTON_IO_48"
+	(global_label "BTN_IOXX"
 		(shape input)
 		(at 142.24 125.73 0)
@@
 		)
 		(property "Intersheetrefs" "${INTERSHEET_REFS}"
-			(at 153.6281 125.73 0)
+			(at 150.493 125.73 0)
 			(effects
 				(font
@@
 		)
 	)
+	(global_label "BTN_IOXY"
+		(shape input)
+		(at 142.24 133.35 0)
+		(fields_autoplaced yes)
+		(effects
+			(font
+				(face "Bahnschrift")
+				(size 1 1)
+				(color 0 0 0 1)
+			)
+			(justify left)
+		)
+		(property "Intersheetrefs" "${INTERSHEET_REFS}"
+			(at 150.4021 133.35 0)
+			(effects
+				(font
+					(size 1.27 1.27)
+				)
+				(justify left)
+				(hide yes)
+			)
+		)
+	)
 	(global_label "BOOT"
 		(shape input)
@@
 		)
 	)
-	(global_label "BUTTON_IO_47"
-		(shape input)
-		(at 142.24 133.35 0)
-		(fields_autoplaced yes)
-		(effects
-			(font
-				(face "Bahnschrift")
-				(size 1 1)
-				(color 0 0 0 1)
-			)
-			(justify left)
-		)
-		(property "Intersheetrefs" "${INTERSHEET_REFS}"
-			(at 153.545 133.35 0)
-			(effects
-				(font
-					(size 1.27 1.27)
-				)
-				(justify left)
-				(hide yes)
-			)
-		)
-	)
-	(global_label "IR MODULE"
+	(global_label "IR_MODULE"
 		(shape passive)
 		(at 170.18 59.69 180)
@@
 		)
 		(property "Intersheetrefs" "${INTERSHEET_REFS}"
-			(at 161.7938 59.69 0)
+			(at 161.5593 59.69 0)
 			(effects
 				(font
@@
 	)
 	(symbol
-		(lib_id "power:+3V3")
-		(at 123.19 125.73 90)
-		(unit 1)
-		(exclude_from_sim no)
-		(in_bom yes)
-		(on_board yes)
-		(dnp no)
-		(property "Reference" "#PWR076"
-			(at 127 125.73 0)
-			(effects
-				(font
-					(size 1.27 1.27)
-				)
-				(hide yes)
-			)
-		)
-		(property "Value" "+3V3"
-			(at 119.38 125.73 90)
-			(effects
-				(font
-					(size 1.27 1.27)
-				)
-				(justify left)
-			)
-		)
-		(property "Footprint" ""
-			(at 123.19 125.73 0)
-			(effects
-				(font
-					(size 1.27 1.27)
-				)
-				(hide yes)
-			)
-		)
-		(property "Datasheet" ""
-			(at 123.19 125.73 0)
-			(effects
-				(font
-					(size 1.27 1.27)
-				)
-				(hide yes)
-			)
-		)
-		(property "Description" ""
-			(at 123.19 125.73 0)
-			(effects
-				(font
-					(size 1.27 1.27)
-				)
-				(hide yes)
-			)
-		)
-		(pin "1"
-		)
-		(instances
-			(project "SUMEC_MK_V"
-				(path "/900bd7ac-cdf9-4a2f-8b1f-2c21e3760046/a907f0f2-2950-481d-8037-7b9f13f2e9c5"
-					(reference "#PWR076")
-					(unit 1)
-				)
-			)
-		)
-	)
-	(symbol
 		(lib_id "Device:C")
 		(at 124.46 109.22 90)
@@
 	(symbol
 		(lib_id "Mechanical:MountingHole_Pad")
-		(at 58.42 52.07 90)
+		(at 58.42 54.61 90)
 		(unit 1)
 		(exclude_from_sim no)
@@
 		(dnp no)
 		(property "Reference" "H4"
-			(at 52.705 52.07 90)
+			(at 52.705 54.61 90)
 			(effects
 				(font
@@
 		)
 		(property "Value" "Mounting Hole M3"
-			(at 57.15 48.26 90)
+			(at 57.15 50.8 90)
 			(effects
 				(font
@@
 		)
 		(property "Footprint" "MountingHole:MountingHole_3.2mm_M3_Pad_Via"
-			(at 58.42 52.07 0)
+			(at 58.42 54.61 0)
 			(effects
 				(font
@@
 		)
 		(property "Datasheet" "~"
-			(at 58.42 52.07 0)
+			(at 58.42 54.61 0)
 			(effects
 				(font
@@
 		)
 		(property "Description" "Mounting Hole with connection"
-			(at 58.42 52.07 0)
+			(at 58.42 54.61 0)
 			(effects
 				(font
@@
 	)
 	(symbol
+		(lib_id "power:GND")
+		(at 124.46 134.62 0)
+		(mirror y)
+		(unit 1)
+		(exclude_from_sim no)
+		(in_bom yes)
+		(on_board yes)
+		(dnp no)
+		(property "Reference" "#PWR083"
+			(at 124.46 140.97 0)
+			(effects
+				(font
+					(size 1.27 1.27)
+				)
+				(hide yes)
+			)
+		)
+		(property "Value" "GND"
+			(at 124.46 138.43 0)
+			(effects
+				(font
+					(size 1.27 1.27)
+				)
+			)
+		)
+		(property "Footprint" ""
+			(at 124.46 134.62 0)
+			(effects
+				(font
+					(size 1.27 1.27)
+				)
+				(hide yes)
+			)
+		)
+		(property "Datasheet" ""
+			(at 124.46 134.62 0)
+			(effects
+				(font
+					(size 1.27 1.27)
+				)
+				(hide yes)
+			)
+		)
+		(property "Description" ""
+			(at 124.46 134.62 0)
+			(effects
+				(font
+					(size 1.27 1.27)
+				)
+				(hide yes)
+			)
+		)
+		(pin "1"
+		)
+		(instances
+			(project "SUMEC_MK_V"
+				(path "/900bd7ac-cdf9-4a2f-8b1f-2c21e3760046/a907f0f2-2950-481d-8037-7b9f13f2e9c5"
+					(reference "#PWR083")
+					(unit 1)
+				)
+			)
+		)
+	)
+	(symbol
 		(lib_id "Connector:TestPoint")
 		(at 158.75 53.34 0)
@@
 	(symbol
 		(lib_id "power:GND")
-		(at 74.93 58.42 0)
+		(at 74.93 57.15 0)
 		(unit 1)
 		(exclude_from_sim no)
@@
 		(dnp no)
 		(property "Reference" "#PWR073"
-			(at 74.93 64.77 0)
+			(at 74.93 63.5 0)
 			(effects
 				(font
@@
 		)
 		(property "Value" "GND"
-			(at 74.93 62.23 0)
+			(at 74.93 60.96 0)
 			(effects
 				(font
@@
 		)
 		(property "Footprint" ""
-			(at 74.93 58.42 0)
+			(at 74.93 57.15 0)
 			(effects
 				(font
@@
 		)
 		(property "Datasheet" ""
-			(at 74.93 58.42 0)
+			(at 74.93 57.15 0)
 			(effects
 				(font
@@
 		)
 		(property "Description" "Power symbol creates a global label with name \"GND\" , ground"
-			(at 74.93 58.42 0)
+			(at 74.93 57.15 0)
 			(effects
 				(font
@@
 	(symbol
 		(lib_id "Mechanical:MountingHole_Pad")
-		(at 58.42 43.18 90)
+		(at 58.42 45.72 90)
 		(unit 1)
 		(exclude_from_sim no)
@@
 		(dnp no)
 		(property "Reference" "H1"
-			(at 52.705 43.18 90)
+			(at 52.705 45.72 90)
 			(effects
 				(font
@@
 		)
 		(property "Value" "Mounting Hole M3"
-			(at 57.15 39.37 90)
+			(at 57.15 41.91 90)
 			(effects
 				(font
@@
 		)
 		(property "Footprint" "MountingHole:MountingHole_3.2mm_M3_Pad_Via"
-			(at 58.42 43.18 0)
+			(at 58.42 45.72 0)
 			(effects
 				(font
@@
 		)
 		(property "Datasheet" "~"
-			(at 58.42 43.18 0)
+			(at 58.42 45.72 0)
 			(effects
 				(font
@@
 		)
 		(property "Description" "Mounting Hole with connection"
-			(at 58.42 43.18 0)
-			(effects
-				(font
+			(at 58.42 45.72 0)
+			(effects
+				(font
