File: main_hw/SUMEC_MK_V/CONNECTIVITY.kicad_sch (KiCad schematic)
At the start: 18 parts, among them J2 USB_TypeC, U3 USBLC6-2SC6

Commit message: MK V Schematic update
Parts:
- added BZ1: Buzzer, Schrack_brd:BUZZER_CUI_CPT, symbol Device:Buzzer
- added R23: 0R, Resistor_SMD:R_0805_2012Metric_Pad1.20x1.40mm_HandSolder, symbol Device:R
Connections:
- net GND: now also BZ1.2 (-)
- new net: BZ1.1 (+), R23.2
- new net BZ1_PWM: R23.1
Other:
- note added: "BUZZER"
- moved on the sheet: C19, C22, D3, D4, D5, D6, D7, F1, J2, R12, R13, R14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

Commit message: Schematic update - finalized
Parts:
- renumbered C19 to C23, C22 to C24, J2 to J4, R12 to R20, R13 to R21, R14 to R22, R16 to R24, R17 to R25, R18 to R26, R19 to R27, R20 to R28, U3 to U5
Connections:
- net VBUS_5V renamed VBUS_USB
Other:
- title: SUMEC_MK_IV -> SUMEC_MK_V
Changed lines of the file:
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@@
 	(paper "A4")
 	(title_block
-		(title "SUMEC_MK_IV")
+		(title "SUMEC_MK_V")
 		(date "2024-08-05")
-		(rev "v3.0.9")
+		(rev "v.1.0.0")
 		(company "SPS NA PROSEKU")
 		(comment 1 "Made in Prague, Czech Republic")
 		(comment 2 "CONTACT: Savva Popov, savva.popov.sp@gmail.com, +420 605 570 366")
 		(comment 3 "Made by bismarx-v1")
-		(comment 4 "SUMEC MK IV aka SMD-V3 board")
+		(comment 4 "SUMEC MK V aka SMD-V4 board")
 	)
 	(rectangle
@@
 		)
 	)
+	(polyline
+		(pts
+			(xy 200.66 82.55) (xy 200.66 69.85)
+		)
+		(stroke
+			(width 0)
+			(type default)
+		)
+	)
 	(wire
 		(pts
@@
 		)
 	)
+	(polyline
+		(pts
+			(xy 213.36 82.55) (xy 200.66 82.55)
+		)
+		(stroke
+			(width 0)
+			(type default)
+		)
+	)
 	(wire
 		(pts
@@
 		)
 	)
+	(polyline
+		(pts
+			(xy 213.36 69.85) (xy 213.36 82.55)
+		)
+		(stroke
+			(width 0)
+			(type default)
+		)
+	)
 	(wire
 		(pts
@@
 		)
 	)
-	(global_label "VBUS_5V"
+	(global_label "VBUS_USB"
 		(shape input)
 		(at 189.23 45.72 0)
@@
 		)
 		(property "Intersheetrefs" "${INTERSHEET_REFS}"
-			(at 197.0619 45.72 0)
+			(at 198.12 45.72 0)
 			(effects
 				(font
@@
 		)
 	)
-	(global_label "VBUS_5V"
+	(global_label "VBUS_USB"
 		(shape output)
 		(at 78.74 36.83 180)
@@
 		)
 		(property "Intersheetrefs" "${INTERSHEET_REFS}"
-			(at 70.9081 36.83 0)
+			(at 69.85 36.83 0)
 			(effects
 				(font
@@
 		(on_board yes)
 		(dnp no)
-		(property "Reference" "#PWR053"
+		(property "Reference" "#PWR064"
 			(at 261.62 62.23 0)
 			(effects
@@
 			(project "SUMEC_MK_V"
 				(path "/900bd7ac-cdf9-4a2f-8b1f-2c21e3760046/ce2ae977-07a3-41c1-b3e1-68b5a1d5517b"
-					(reference "#PWR053")
+					(reference "#PWR064")
 					(unit 1)
 				)
@@
 		(on_board yes)
 		(dnp no)
-		(property "Reference" "R20"
+		(property "Reference" "R28"
 			(at 253.365 59.055 90)
 			(effects
@@
 			(project "SUMEC_MK_V"
 				(path "/900bd7ac-cdf9-4a2f-8b1f-2c21e3760046/ce2ae977-07a3-41c1-b3e1-68b5a1d5517b"
-					(reference "R20")
+					(reference "R28")
 					(unit 1)
 				)
@@
 		(on_board yes)
 		(dnp no)
-		(property "Reference" "R16"
+		(property "Reference" "R24"
 			(at 252.73 28.575 90)
 			(effects
@@
 			(project "SUMEC_MK_V"
 				(path "/900bd7ac-cdf9-4a2f-8b1f-2c21e3760046/ce2ae977-07a3-41c1-b3e1-68b5a1d5517b"
-					(reference "R16")
+					(reference "R24")
 					(unit 1)
 				)
@@
 		(on_board yes)
 		(dnp no)
-		(property "Reference" "#PWR050"
+		(property "Reference" "#PWR061"
 			(at 261.62 39.37 0)
 			(effects
@@
 			(project "SUMEC_MK_V"
 				(path "/900bd7ac-cdf9-4a2f-8b1f-2c21e3760046/ce2ae977-07a3-41c1-b3e1-68b5a1d5517b"
-					(reference "#PWR050")
+					(reference "#PWR061")
 					(unit 1)
 				)
@@
 		(on_board yes)
 		(dnp no)
-		(property "Reference" "R17"
+		(property "Reference" "R25"
 			(at 252.73 36.195 90)
 			(effects
@@
 			(project "SUMEC_MK_V"
 				(path "/900bd7ac-cdf9-4a2f-8b1f-2c21e3760046/ce2ae977-07a3-41c1-b3e1-68b5a1d5517b"
-					(reference "R17")
+					(reference "R25")
 					(unit 1)
 				)
@@
 		(dnp no)
 		(fields_autoplaced yes)
-		(property "Reference" "#PWR040"
+		(property "Reference" "#PWR057"
 			(at 138.43 45.72 0)
 			(effects
@@
 			(project "SUMEC_MK_V"
 				(path "/900bd7ac-cdf9-4a2f-8b1f-2c21e3760046/ce2ae977-07a3-41c1-b3e1-68b5a1d5517b"
-					(reference "#PWR040")
+					(reference "#PWR057")
 					(unit 1)
 				)
@@
 		(on_board yes)
 		(dnp no)
-		(property "Reference" "#PWR051"
+		(property "Reference" "#PWR062"
 			(at 261.62 46.99 0)
 			(effects
@@
 			(project "SUMEC_MK_V"
 				(path "/900bd7ac-cdf9-4a2f-8b1f-2c21e3760046/ce2ae977-07a3-41c1-b3e1-68b5a1d5517b"
-					(reference "#PWR051")
+					(reference "#PWR062")
 					(unit 1)
 				)
@@
 		(dnp no)
 		(fields_autoplaced yes)
-		(property "Reference" "#PWR0102"
+		(property "Reference" "#PWR060"
 			(at 245.11 118.11 0)
 			(effects
@@
 			(project "SUMEC_MK_V"
 				(path "/900bd7ac-cdf9-4a2f-8b1f-2c21e3760046/ce2ae977-07a3-41c1-b3e1-68b5a1d5517b"
-					(reference "#PWR0102")
+					(reference "#PWR060")
 					(unit 1)
 				)
@@
 		(on_board yes)
 		(dnp no)
-		(property "Reference" "R18"
+		(property "Reference" "R26"
 			(at 253.365 43.815 90)
 			(effects
@@
 			(project "SUMEC_MK_V"
 				(path "/900bd7ac-cdf9-4a2f-8b1f-2c21e3760046/ce2ae977-07a3-41c1-b3e1-68b5a1d5517b"
-					(reference "R18")
+					(reference "R26")
 					(unit 1)
 				)
@@
 		(on_board yes)
 		(dnp no)
-		(property "Reference" "#PWR054"
+		(property "Reference" "#PWR065"
 			(at 261.62 69.85 0)
 			(effects
@@
 			(project "SUMEC_MK_V"
 				(path "/900bd7ac-cdf9-4a2f-8b1f-2c21e3760046/ce2ae977-07a3-41c1-b3e1-68b5a1d5517b"
-					(reference "#PWR054")
+					(reference "#PWR065")
 					(unit 1)
 				)
@@
 		(on_board yes)
 		(dnp no)
-		(property "Reference" "R14"
+		(property "Reference" "R22"
 			(at 139.065 53.975 90)
 			(effects
@@
 			(project "SUMEC_MK_V"
 				(path "/900bd7ac-cdf9-4a2f-8b1f-2c21e3760046/ce2ae977-07a3-41c1-b3e1-68b5a1d5517b"
-					(reference "R14")
+					(reference "R22")
 					(unit 1)
 				)
@@
 		(dnp no)
 		(fields_autoplaced yes)
-		(property "Reference" "#PWR039"
+		(property "Reference" "#PWR056"
 			(at 93.98 68.58 0)
 			(effects
@@
 			(project "SUMEC_MK_V"
 				(path "/900bd7ac-cdf9-4a2f-8b1f-2c21e3760046/ce2ae977-07a3-41c1-b3e1-68b5a1d5517b"
-					(reference "#PWR039")
+					(reference "#PWR056")
 					(unit 1)
 				)
@@
 		(on_board yes)
 		(dnp no)
-		(property "Reference" "R13"
+		(property "Reference" "R21"
 			(at 139.065 28.575 90)
 			(effects
@@
 			(project "SUMEC_MK_V"
 				(path "/900bd7ac-cdf9-4a2f-8b1f-2c21e3760046/ce2ae977-07a3-41c1-b3e1-68b5a1d5517b"
-					(reference "R13")
+					(reference "R21")
 					(unit 1)
 				)
@@
 		(dnp no)
 		(fields_autoplaced yes)
-		(property "Reference" "#PWR044"
+		(property "Reference" "#PWR058"
 			(at 187.96 59.69 0)
 			(effects
@@
 			(project "SUMEC_MK_V"
 				(path "/900bd7ac-cdf9-4a2f-8b1f-2c21e3760046/ce2ae977-07a3-41c1-b3e1-68b5a1d5517b"
-					(reference "#PWR044")
+					(reference "#PWR058")
 					(unit 1)
 				)
@@
 		(on_board yes)
 		(dnp no)
-		(property "Reference" "#PWR046"
+		(property "Reference" "#PWR059"
 			(at 236.22 33.02 0)
 			(effects
@@
 			(project "SUMEC_MK_V"
 				(path "/900bd7ac-cdf9-4a2f-8b1f-2c21e3760046/ce2ae977-07a3-41c1-b3e1-68b5a1d5517b"
-					(reference "#PWR046")
+					(reference "#PWR059")
 					(unit 1)
 				)
@@
 		(on_board yes)
 		(dnp no)
-		(property "Reference" "C22"
+		(property "Reference" "C24"
 			(at 190.5 48.895 0)
 			(effects
@@
 			(project "SUMEC_MK_V"
 				(path "/900bd7ac-cdf9-4a2f-8b1f-2c21e3760046/ce2ae977-07a3-41c1-b3e1-68b5a1d5517b"
-					(reference "C22")
+					(reference "C24")
 					(unit 1)
 				)
@@
 		(on_board yes)
 		(dnp no)
-		(property "Reference" "C19"
+		(property "Reference" "C23"
 			(at 82.804 57.15 0)
 			(effects
@@
 			(project "SUMEC_MK_V"
 				(path "/900bd7ac-cdf9-4a2f-8b1f-2c21e3760046/ce2ae977-07a3-41c1-b3e1-68b5a1d5517b"
-					(reference "C19")
+					(reference "C23")
 					(unit 1)
 				)
@@
 		(on_board yes)
 		(dnp no)
-		(property "Reference" "#PWR052"
+		(property "Reference" "#PWR063"
 			(at 261.62 54.61 0)
 			(effects
@@
 			(project "SUMEC_MK_V"
 				(path "/900bd7ac-cdf9-4a2f-8b1f-2c21e3760046/ce2ae977-07a3-41c1-b3e1-68b5a1d5517b"
-					(reference "#PWR052")
+					(reference "#PWR063")
 					(unit 1)
 				)
@@
 		(on_board yes)
 		(dnp no)
-		(property "Reference" "J2"
+		(property "Reference" "J4"
 			(at 111.76 29.845 0)
 			(effects
@@
 			(project "SUMEC_MK_V"
 				(path "/900bd7ac-cdf9-4a2f-8b1f-2c21e3760046/ce2ae977-07a3-41c1-b3e1-68b5a1d5517b"
-					(reference "J2")
+					(reference "J4")
 					(unit 1)
 				)
@@
 		(dnp no)
 		(fields_autoplaced yes)
-		(property "Reference" "U3"
+		(property "Reference" "U5"
 			(at 166.37 26.67 0)
 			(effects
@@
 			(project "SUMEC_MK_V"
 				(path "/900bd7ac-cdf9-4a2f-8b1f-2c21e3760046/ce2ae977-07a3-41c1-b3e1-68b5a1d5517b"
-					(reference "U3")
+					(reference "U5")
 					(unit 1)
 				)
@@
 		(on_board yes)
 		(dnp no)
-		(property "Reference" "R12"
+		(property "Reference" "R20"
 			(at 75.184 57.15 0)
 			(effects
@@
 			(project "SUMEC_MK_V"
 				(path "/900bd7ac-cdf9-4a2f-8b1f-2c21e3760046/ce2ae977-07a3-41c1-b3e1-68b5a1d5517b"
-					(reference "R12")
+					(reference "R20")
 					(unit 1)
 				)
@@
 		(on_board yes)
 		(dnp no)
-		(property "Reference" "R19"
+		(property "Reference" "R27"
 			(at 253.365 51.435 90)
 			(effects
@@
 			(project "SUMEC_MK_V"
 				(path "/900bd7ac-cdf9-4a2f-8b1f-2c21e3760046/ce2ae977-07a3-41c1-b3e1-68b5a1d5517b"
-					(reference "R19")
+					(reference "R27")
 					(unit 1)
 				)

Commit message: MK V Schematic update
Parts:
- renumbered C23 to C27, C24 to C28, R20 to R24, R22 to R25, R21 to R26, R23 to R27, R24 to R28, R25 to R29, R26 to R30, R27 to R31, R28 to R32, U5 to U6
Connections:
- net D+: now also U6.4; no longer U6.6
- net D-: now also U6.6; no longer U6.4
- net at R25.2: now also U6.1; no longer U6.3
- net at R26.2: now also U6.3; no longer U6.1
Other:
- moved on the sheet: R25, R26

Commit message: PCB update MKV
Connections:
- net GND: now also D4.1 (K); no longer R29.2
- net VBUS_USB: now also R29.1
- net VBUS 5V: no longer names the net of D4.2 (A)
- net VBUS 5V: now also R29.2
Other:
- moved on the sheet: D4, R29
Changed lines of the file:
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@@
+		)
+	)
+	(global_label "VBUS_USB"
+		(shape input)
+		(at 232.41 40.64 180)
+		(fields_autoplaced yes)
+		(effects
+			(font
+				(face "Bahnschrift")
+				(size 1 1)
+				(color 0 0 0 1)
+			)
+			(justify right)
+		)
+		(property "Intersheetrefs" "${INTERSHEET_REFS}"
+			(at 223.52 40.64 0)
+			(effects
+				(font
+					(size 1.27 1.27)
+				)
+				(justify right)
+				(hide yes)
+			)
 		)
 	)
@@
 		)
 	)
-	(global_label "VBUS 5V"
-		(shape input)
-		(at 232.41 40.64 180)
-		(fields_autoplaced yes)
-		(effects
-			(font
-				(face "Bahnschrift")
-				(size 1 1)
-				(color 0 0 0 1)
-			)
-			(justify right)
-		)
-		(property "Intersheetrefs" "${INTERSHEET_REFS}"
-			(at 224.8126 40.64 0)
-			(effects
-				(font
-					(size 1.27 1.27)
-				)
-				(justify right)
-				(hide yes)
-			)
-		)
-	)
 	(global_label "D_NEG_IN"
 		(shape input)
@@
 	(symbol
 		(lib_id "Device:R")
-		(at 251.46 40.64 90)
+		(at 240.03 40.64 90)
 		(unit 1)
 		(exclude_from_sim no)
@@
 		(dnp no)
 		(property "Reference" "R29"
-			(at 252.73 36.195 90)
+			(at 241.3 36.195 90)
 			(effects
 				(font
@@
 		)
 		(property "Value" "220R"
-			(at 254 38.1 90)
+			(at 242.57 38.1 90)
 			(effects
 				(font
@@
 		)
 		(property "Footprint" "Resistor_SMD:R_0805_2012Metric_Pad1.20x1.40mm_HandSolder"
-			(at 251.46 42.418 90)
+			(at 240.03 42.418 90)
 			(effects
 				(font
@@
 		)
 		(property "Datasheet" "~"
-			(at 251.46 40.64 0)
+			(at 240.03 40.64 0)
 			(effects
 				(font
@@
 		)
 		(property "Description" ""
-			(at 251.46 40.64 0)
+			(at 240.03 40.64 0)
 			(effects
 				(font
@@
 	(symbol
 		(lib_id "Device:LED")
-		(at 240.03 40.64 180)
+		(at 251.46 40.64 180)
 		(unit 1)
 		(exclude_from_sim no)
@@
 		(dnp no)
 		(property "Reference" "D4"
-			(at 238.125 36.195 0)
+			(at 249.555 36.195 0)
 			(effects
 				(font
@@
 		)
 		(property "Value" "LED"
-			(at 238.125 38.1 0)
+			(at 249.555 38.1 0)
 			(effects
 				(font
@@
 		)
 		(property "Footprint" "LED_SMD:LED_0805_2012Metric_Pad1.15x1.40mm_HandSolder"
-			(at 240.03 40.64 0)
+			(at 251.46 40.64 0)
 			(effects
 				(font
@@
 		)
 		(property "Datasheet" "~"
-			(at 240.03 40.64 0)
+			(at 251.46 40.64 0)
 			(effects
 				(font
@@
 		)
 		(property "Description" ""
-			(at 240.03 40.64 0)
-			(effects
-				(font
+			(at 251.46 40.64 0)
+			(effects
+				(font

Commit message: pcb update
Parts:
- R28: value 1000k -> 1k
Connections:
- net GND: now also D5.1 (K), D6.1 (K), D7.1 (K); no longer R30.2, R31.2, R32.2
- net LED_1: now also R30.1; no longer D5.2 (A)
- net LED_2: now also R31.1; no longer D6.2 (A)
- net LED_3: now also R32.1; no longer D7.2 (A)
- new net: D7.2 (A), R32.2
- new net: D5.2 (A), R30.2
- new net: D6.2 (A), R31.2
Other:
- moved on the sheet: D5, D6, D7, R30, R31, R32

Commit message: PCB routing update
Connections:
- net +12V: now also R28.1; no longer D3.2 (A)
- net GND: now also D3.1 (K); no longer R28.2
- new net: D3.2 (A), R28.2
Other:
- moved on the sheet: D3, R28
Changed lines of the file:
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@@
 	(symbol
 		(lib_id "Device:R")
-		(at 251.46 33.02 90)
+		(at 240.03 33.02 90)
 		(unit 1)
 		(exclude_from_sim no)
@@
 		(dnp no)
 		(property "Reference" "R28"
-			(at 252.73 28.575 90)
+			(at 241.3 28.575 90)
 			(effects
 				(font
@@
 		)
 		(property "Value" "1k"
-			(at 251.46 30.48 90)
+			(at 240.03 30.48 90)
 			(effects
 				(font
@@
 		)
 		(property "Footprint" "Resistor_SMD:R_0805_2012Metric_Pad1.20x1.40mm_HandSolder"
-			(at 251.46 34.798 90)
+			(at 240.03 34.798 90)
 			(effects
 				(font
@@
 		)
 		(property "Datasheet" "~"
-			(at 251.46 33.02 0)
-			(effects
-				(font
-					(size 1.27 1.27)
-				)
-				(hide yes)
-			)
-		)
-		(property "Description" ""
-			(at 251.46 33.02 0)
+			(at 240.03 33.02 0)
+			(effects
+				(font
+					(size 1.27 1.27)
+				)
+				(hide yes)
+			)
+		)
+		(property "Description" ""
+			(at 240.03 33.02 0)
 			(effects
 				(font
@@
 	(symbol
 		(lib_id "Device:LED")
-		(at 240.03 33.02 180)
+		(at 251.46 33.02 180)
 		(unit 1)
 		(exclude_from_sim no)
@@
 		(dnp no)
 		(property "Reference" "D3"
-			(at 238.125 28.575 0)
+			(at 249.555 28.575 0)
 			(effects
 				(font
@@
 		)
 		(property "Value" "LED"
-			(at 238.125 30.48 0)
+			(at 249.555 30.48 0)
 			(effects
 				(font
@@
 		)
 		(property "Footprint" "LED_SMD:LED_0805_2012Metric_Pad1.15x1.40mm_HandSolder"
-			(at 240.03 33.02 0)
+			(at 251.46 33.02 0)
 			(effects
 				(font
@@
 		)
 		(property "Datasheet" "~"
-			(at 240.03 33.02 0)
-			(effects
-				(font
-					(size 1.27 1.27)
-				)
-				(hide yes)
-			)
-		)
-		(property "Description" ""
-			(at 240.03 33.02 0)
-			(effects
-				(font
+			(at 251.46 33.02 0)
+			(effects
+				(font
+					(size 1.27 1.27)
+				)
+				(hide yes)
+			)
+		)
+		(property "Description" ""
+			(at 251.46 33.02 0)
+			(effects
+				(font
