File: main_hw/SUMEC_MK_V/SUMEC_MK_V.kicad_sch (KiCad schematic)
At the start: 13 parts, among them J15 39502-1009, J16 39502-1009, U5 TBA2-0511, U6 NCP1117-3.3

Commit message: MK V Schematic update
Connections:
- no-connect marks 2 -> 1
Other:
- note added: "1. Q: Gyro+accelometer - possible to add 2. Q: Passive buzzer 3. Q: Left/right silk for sensors and motors 4. Q: External eeprom - 1kb max 5. Q: Add IO pin numbers after the routing is done 6. Q: VBATT voltage read 7. Q: Ferrite bead for USB"
- note added: "GRAPHICS"
- note removed: "1. Q: Gyro+accelometer - possible to add 2. Q: Passive buzzer 3. Q: Left/right silk for sensors and motors 4. Q: External eeprom? FRAM? 5. Q: Add IO pin numbers after the routing is done 6. Q: VBATT voltage read"
- note removed: "ART"
- moved on the sheet: C27, C28, C29, J15, J16, U5, U6

Commit message: Schematic update - finalized
Parts:
- removed C27: 22uF, Capacitor_SMD:C_0805_2012Metric_Pad1.18x1.45mm_HandSolder, symbol Device:C_Polarized
- removed C28, C29: 10uF, Capacitor_Tantalum_SMD:CP_EIA-3216-18_Kemet-A_Pad1.58x1.35mm_HandSolder, symbol Device:C_Polarized
- removed J15, J16: 39502-1009, IoTGW:Molex_9pin_3.50, symbol Connector:Conn_01x09_Socket
- removed U5: TBA2-0511, Converter_DCDC:Converter_DCDC_TRACO_TBA2-xxxx_Single_THT, symbol Converter_DCDC:TBA2-0511
- removed U6: NCP1117-3.3, Package_TO_SOT_SMD:SOT-223-3_TabPin2, symbol Regulator_Linear:NCP1117-3.3_SOT223
- TP1: renamed from TP6; footprint sumec_graphic:SPS_LOGO_IMG -> (none)
- TP2: renamed from TP7; footprint sumec_graphic:SUMEC_LOGO_IMG -> (none)
- TP3: renamed from TP8; footprint sumec_graphic:ULTRAKILL_IMG -> (none)
- TP4: renamed from TP9; footprint sumec_graphic:SUMEC_QR_IMG -> (none)
- TP5: renamed from TP10; footprint sumec_graphic:FREEFALL2_IMG -> (none)
- TP6: renamed from TP11; footprint sumec_graphic:ME_FR_IMG -> (none)
Connections:
- no-connect marks 1 -> 0
Other:
- note added: "1. Q: 2. Q: 3. Q: Left/right silk for sensors and motors 4. Q: 5. Q: Add IO pin numbers after the routing is done 6. Q: 7. Q:"
- note removed: "1. Q: Gyro+accelometer - possible to add 2. Q: Passive buzzer 3. Q: Left/right silk for sensors and motors 4. Q: External eeprom - 1kb max 5. Q: Add IO pin numbers after the routing is done 6. Q: VBATT voltage read 7. Q: Ferrite bead for USB"
- note removed: "105,50CZK"
- note removed: "11,53CZK"
- note removed: "42,35CZK"
- note removed: "43,86CZK"
- note removed: "CONNECTORS"
- note removed: "F"
- note removed: "Isolation: 1.5kV Output current: 400mA Output voltage: 5V Input voltage: 4.5V-5.5V Output power: 2W BUILT IN SHORT CIRCUIT PROTECTION"
- note removed: "LDO. VOLTAGE REG."
- note removed: "M"
- note removed: "Molex 9Pin header, 3.5mm Plug (female conn): 39503-3009"
- note removed: "Output voltage: 3.3V Output current: 1A Max Input voltage: 12V Quiescent Current: 6mA"
- note removed: "POWER ISOLATION"
- title: SUMEC_MK_IV -> SUMEC_MK_V

Commit message: MK V Schematic update
Other:
- note added: "1. Q: 2. Q: 3. Q: Left/right silk for sensors and motors 4. Q: 5. Q: Add IO pin numbers after the routing is done 6. Q: Does the voltage read need to be after the switch or before? 7. Q:"
- note removed: "1. Q: 2. Q: 3. Q: Left/right silk for sensors and motors 4. Q: 5. Q: Add IO pin numbers after the routing is done 6. Q: 7. Q:"
Changed lines of the file:
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@@
 		)
 	)
-	(text "1. Q: \n2. Q: \n3. Q: Left/right silk for sensors and motors\n4. Q: \n5. Q: Add IO pin numbers after the routing is done\n6. Q: \n7. Q: "
+	(text "1. Q: \n2. Q: \n3. Q: Left/right silk for sensors and motors\n4. Q: \n5. Q: Add IO pin numbers after the routing is done\n6. Q: Does the voltage read need to be after the switch or before?\n7. Q: "
 		(exclude_from_sim no)
 		(at 20.32 183.134 0)
@@
 				(effects
 					(font
+						(face "Bahnschrift")
+						(size 1 1)
+						(bold yes)
+						(italic yes)
+						(color 0 0 0 1)
+					)
+					(justify left top)
+				)
+			)
+			(table_cell "I2C ADRRESS"
+				(exclude_from_sim no)
+				(at 116.205 170.18 0)
+				(size 19.685 2.54)
+				(margins 0.9525 0.9525 0.9525 0.9525)
+				(span 1 1)
+				(fill
+					(type none)
+				)
+				(effects
+					(font
+						(face "Bahnschrift")
+						(size 1 1)
+						(bold yes)
+						(italic yes)
+						(color 0 0 0 1)
+					)
+					(justify left top)
+				)
+			)
+			(table_cell "GYROSCOPE - BMI088"
+				(exclude_from_sim no)
+				(at 96.52 172.72 0)
+				(size 19.685 2.54)
+				(margins 0.9525 0.9525 0.9525 0.9525)
+				(span 1 1)
+				(fill
+					(type none)
+				)
+				(effects
+					(font
+						(face "Bahnschrift")
+						(size 1 1)
+						(color 0 0 0 1)
+					)
+					(justify left top)
+				)
+			)
+			(table_cell "0x69"
+				(exclude_from_sim no)
+				(at 116.205 172.72 0)
+				(size 19.685 2.54)
+				(margins 0.9525 0.9525 0.9525 0.9525)
+				(span 1 1)
+				(fill
+					(type none)
+				)
+				(effects
+					(font
+						(face "Bahnschrift")
 						(size 1.27 1.27)
-					)
-					(justify left top)
-				)
-			)
-			(table_cell "I2C ADRRESS"
-				(exclude_from_sim no)
-				(at 116.205 170.18 0)
-				(size 19.685 2.54)
-				(margins 0.9525 0.9525 0.9525 0.9525)
-				(span 1 1)
-				(fill
-					(type none)
-				)
-				(effects
-					(font
+						(color 0 0 0 1)
+					)
+					(justify left top)
+				)
+			)
+			(table_cell "ACCELEROMETER - BMI088"
+				(exclude_from_sim no)
+				(at 96.52 175.26 0)
+				(size 19.685 2.54)
+				(margins 0.9525 0.9525 0.9525 0.9525)
+				(span 1 1)
+				(fill
+					(type none)
+				)
+				(effects
+					(font
+						(face "Bahnschrift")
+						(size 1 1)
+						(color 0 0 0 1)
+					)
+					(justify left top)
+				)
+			)
+			(table_cell "0x19"
+				(exclude_from_sim no)
+				(at 116.205 175.26 0)
+				(size 19.685 2.54)
+				(margins 0.9525 0.9525 0.9525 0.9525)
+				(span 1 1)
+				(fill
+					(type none)
+				)
+				(effects
+					(font
+						(face "Bahnschrift")
 						(size 1.27 1.27)
-					)
-					(justify left top)
-				)
-			)
-			(table_cell "GYROSCOPE"
-				(exclude_from_sim no)
-				(at 96.52 172.72 0)
-				(size 19.685 2.54)
-				(margins 0.9525 0.9525 0.9525 0.9525)
-				(span 1 1)
-				(fill
-					(type none)
-				)
-				(effects
-					(font
+						(color 0 0 0 1)
+					)
+					(justify left top)
+				)
+			)
+			(table_cell "EEPROM - 24CW1280T"
+				(exclude_from_sim no)
+				(at 96.52 177.8 0)
+				(size 19.685 2.54)
+				(margins 0.9525 0.9525 0.9525 0.9525)
+				(span 1 1)
+				(fill
+					(type none)
+				)
+				(effects
+					(font
+						(face "Bahnschrift")
+						(size 1 1)
+						(color 0 0 0 1)
+					)
+					(justify left top)
+				)
+			)
+			(table_cell "0x50"
+				(exclude_from_sim no)
+				(at 116.205 177.8 0)
+				(size 19.685 2.54)
+				(margins 0.9525 0.9525 0.9525 0.9525)
+				(span 1 1)
+				(fill
+					(type none)
+				)
+				(effects
+					(font
+						(face "Bahnschrift")
 						(size 1.27 1.27)
-					)
-					(justify left top)
-				)
-			)
-			(table_cell ""
-				(exclude_from_sim no)
-				(at 116.205 172.72 0)
-				(size 19.685 2.54)
-				(margins 0.9525 0.9525 0.9525 0.9525)
-				(span 1 1)
-				(fill
-					(type none)
-				)
-				(effects
-					(font
+						(color 0 0 0 1)
+					)
+					(justify left top)
+				)
+			)
+			(table_cell "VOLTAGE READ - INU226"
+				(exclude_from_sim no)
+				(at 96.52 180.34 0)
+				(size 19.685 2.54)
+				(margins 0.9525 0.9525 0.9525 0.9525)
+				(span 1 1)
+				(fill
+					(type none)
+				)
+				(effects
+					(font
+						(face "Bahnschrift")
+						(size 1 1)
+						(color 0 0 0 1)
+					)
+					(justify left top)
+				)
+			)
+			(table_cell "0x40"
+				(exclude_from_sim no)
+				(at 116.205 180.34 0)
+				(size 19.685 2.54)
+				(margins 0.9525 0.9525 0.9525 0.9525)
+				(span 1 1)
+				(fill
+					(type none)
+				)
+				(effects
+					(font
+						(face "Bahnschrift")
 						(size 1.27 1.27)
-					)
-					(justify left top)
-				)
-			)
-			(table_cell "ACCELEROMETER"
-				(exclude_from_sim no)
-				(at 96.52 175.26 0)
-				(size 19.685 2.54)
-				(margins 0.9525 0.9525 0.9525 0.9525)
-				(span 1 1)
-				(fill
-					(type none)
-				)
-				(effects
-					(font
-						(size 1.27 1.27)
-					)
-					(justify left top)
-				)
-			)
-			(table_cell ""
-				(exclude_from_sim no)
-				(at 116.205 175.26 0)
-				(size 19.685 2.54)
-				(margins 0.9525 0.9525 0.9525 0.9525)
-				(span 1 1)
-				(fill
-					(type none)
-				)
-				(effects
-					(font
-						(size 1.27 1.27)
-					)
-					(justify left top)
-				)
-			)
-			(table_cell "EEPROM"
-				(exclude_from_sim no)
-				(at 96.52 177.8 0)
-				(size 19.685 2.54)
-				(margins 0.9525 0.9525 0.9525 0.9525)
-				(span 1 1)
-				(fill
-					(type none)
-				)
-				(effects
-					(font
-						(size 1.27 1.27)
-					)
-					(justify left top)
-				)
-			)
-			(table_cell ""
-				(exclude_from_sim no)
-				(at 116.205 177.8 0)
-				(size 19.685 2.54)
-				(margins 0.9525 0.9525 0.9525 0.9525)
-				(span 1 1)
-				(fill
-					(type none)
-				)
-				(effects
-					(font
-						(size 1.27 1.27)
-					)
-					(justify left top)
-				)
-			)
-			(table_cell "BMI008"
-				(exclude_from_sim no)
-				(at 96.52 180.34 0)
-				(size 19.685 2.54)
-				(margins 0.9525 0.9525 0.9525 0.9525)
-				(span 1 1)
-				(fill
-					(type none)
-				)
-				(effects
-					(font
-						(size 1.27 1.27)
-					)
-					(justify left top)
-				)
-			)
-			(table_cell ""
-				(exclude_from_sim no)
-				(at 116.205 180.34 0)
-				(size 19.685 2.54)
-				(margins 0.9525 0.9525 0.9525 0.9525)
-				(span 1 1)
-				(fill
-					(type none)
-				)
-				(effects
-					(font
-						(size 1.27 1.27)
-					)
-					(justify left top)
+						(color 0 0 0 1)
+					)
+					(justify left top)

Commit message: PCB Updtae MK5
Changed lines of the file:
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@@
-		)
-	)
-	(bus
-		(pts
-			(xy 187.96 105.41) (xy 187.96 96.52)
-		)
-		(stroke
-			(width 0)
-			(type default)
-		)
-	)
-	(bus
-		(pts
-			(xy 179.07 105.41) (xy 179.07 96.52)
-		)
-		(stroke
-			(width 0)
-			(type default)
-		)
-	)
-	(bus
-		(pts
-			(xy 110.49 105.41) (xy 110.49 96.52)
-		)
-		(stroke
-			(width 0)
-			(type default)
 		)
 	)
@@
 		(pts
 			(xy 153.67 191.77) (xy 153.67 189.23)
-		)
-		(stroke
-			(width 0)
-			(type default)
-		)
-	)
-	(bus
-		(pts
-			(xy 50.8 96.52) (xy 110.49 96.52)
 		)
 		(stroke
@@
 		)
 	)
-	(bus
-		(pts
-			(xy 119.38 96.52) (xy 179.07 96.52)
-		)
-		(stroke
-			(width 0)
-			(type default)
-		)
-	)
 	(wire
 		(pts
 			(xy 165.1 191.77) (xy 165.1 189.23)
-		)
-		(stroke
-			(width 0)
-			(type default)
-		)
-	)
-	(bus
-		(pts
-			(xy 187.96 105.41) (xy 179.07 105.41)
 		)
 		(stroke
@@
 		)
 		(stroke
-			(width 0)
-			(type default)
-		)
-	)
-	(bus
-		(pts
-			(xy 119.38 105.41) (xy 110.49 105.41)
-		)
-		(stroke
-			(width 0)
-			(type default)
-		)
-	)
-	(bus
-		(pts
-			(xy 119.38 105.41) (xy 119.38 96.52)
-		)
-		(stroke
-			(width 0)
-			(type default)
-		)
-	)
-	(bus
-		(pts
-			(xy 187.96 96.52) (xy 247.65 96.52)
-		)
-		(stroke

Commit message: a lot of routing and layout updates
Other:
- sheet MOTOR_CONTROL renamed MOTOR CONTROL
- sheet POWER_SUPPLY renamed POWER
Changed lines of the file:
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@@
 			(color 255 255 255 1.0000)
 		)
-		(property "Sheetname" "MOTOR_CONTROL"
-			(at 147.955 81.28 0)
+		(property "Sheetname" "MOTOR CONTROL"
+			(at 149.225 80.645 0)
 			(effects
 				(font
@@
 			(color 255 255 255 1.0000)
 		)
-		(property "Sheetname" "POWER_SUPPLY"
+		(property "Sheetname" "POWER"
 			(at 79.375 81.28 0)
 			(effects

Commit message: SUMEC MKIV
Parts:
- TP6: footprint (none) -> sumec_graphic:CALIPER_IMG
Other:
- note added: "CALIPER-KARNIK"
- note removed: "ME FR"
Changed lines of the file:
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@@
 		)
 	)
-	(text "ME FR"
+	(text "CALIPER-KARNIK"
 		(exclude_from_sim no)
 		(at 169.545 184.15 90)
@@
 			)
 		)
-		(property "Footprint" ""
+		(property "Footprint" "sumec_graphic:CALIPER_IMG"
 			(at 173.99 189.23 0)
 			(effects

Commit message: new qre board
Parts:
- added TP19: TestPoint, sumec_graphic:SUMEC_QR_IMG, symbol Connector:TestPoint
- added TP20: TestPoint, sumec_graphic:BEE_IMG, symbol Connector:TestPoint
- added TP21: TestPoint, sumec_graphic:FLOWER_IMG, symbol Connector:TestPoint
- added TP22: TestPoint, sumec_graphic:SYMBOL_IMG, symbol Connector:TestPoint
- TP1: footprint (none) -> sumec_graphic:SPS_LOGO_IMG
- TP2: footprint (none) -> sumec_graphic:SUMEC_LOGO_IMG
- TP3: footprint (none) -> sumec_graphic:CATTO_MASK_IMG
- TP4: footprint (none) -> sumec_graphic:OWO_WHATS_THIS_IMG
- TP5: footprint (none) -> sumec_graphic:HANKA_THINGY_IMG
Connections:
- net at TP1.1, TP2.1, TP3.1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: now also TP19.1, TP20.1, TP21.1, TP22.1
Other:
- note added: "BEE"
- note added: "CATTO"
- note added: "FLOWER"
- note added: "HANKA THINGY"
- note added: "OWO WHATS THIS"
- note added: "SUMEC QR"
- note added: "SYMBOL"
- note removed: "FREEFALL PANEL"
- note removed: "SUMEC LINKTREE"
- note removed: "ULTRAKILL V1"
