File: main_hw/SUMEC_MK_V/MCU.kicad_sch (KiCad schematic)
At the start: 7 parts, among them U3 ESP32-S3-WROOM-1, U4 24CW1280T-I/OT

Commit message: updates to mk5
Parts:
- renumbered C21 to C20, C22 to C21, C23 to C22, R12 to R11, R13 to R12, U4 to U3, U3 to U4
Changed lines of the file:
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@@
 		(on_board yes)
 		(dnp no)
-		(property "Reference" "#PWR054"
+		(property "Reference" "#PWR051"
 			(at 80.01 142.24 0)
 			(effects
@@
 			(project "SUMEC_MK_V"
 				(path "/900bd7ac-cdf9-4a2f-8b1f-2c21e3760046/7b93d7c5-db1a-415c-92e4-9ebec6cf195f"
-					(reference "#PWR054")
+					(reference "#PWR051")
 					(unit 1)
 				)
@@
 		(dnp no)
 		(fields_autoplaced yes)
-		(property "Reference" "U4"
+		(property "Reference" "U3"
 			(at 92.3133 137.16 0)
 			(effects
@@
 			(project "SUMEC_MK_V"
 				(path "/900bd7ac-cdf9-4a2f-8b1f-2c21e3760046/7b93d7c5-db1a-415c-92e4-9ebec6cf195f"
-					(reference "U4")
+					(reference "U3")
 					(unit 1)
 				)
@@
 		(on_board yes)
 		(dnp no)
-		(property "Reference" "#PWR061"
+		(property "Reference" "#PWR058"
 			(at 226.06 82.55 0)
 			(effects
@@
 			(project "SUMEC_MK_V"
 				(path "/900bd7ac-cdf9-4a2f-8b1f-2c21e3760046/7b93d7c5-db1a-415c-92e4-9ebec6cf195f"
-					(reference "#PWR061")
+					(reference "#PWR058")
 					(unit 1)
 				)
@@
 		(on_board yes)
 		(dnp no)
-		(property "Reference" "#PWR060"
+		(property "Reference" "#PWR057"
 			(at 218.44 82.55 0)
 			(effects
@@
 			(project "SUMEC_MK_V"
 				(path "/900bd7ac-cdf9-4a2f-8b1f-2c21e3760046/7b93d7c5-db1a-415c-92e4-9ebec6cf195f"
-					(reference "#PWR060")
+					(reference "#PWR057")
 					(unit 1)
 				)
@@
 		(on_board yes)
 		(dnp no)
-		(property "Reference" "R12"
+		(property "Reference" "R11"
 			(at 215.265 83.82 0)
 			(effects
@@
 			(project "SUMEC_MK_V"
 				(path "/900bd7ac-cdf9-4a2f-8b1f-2c21e3760046/7b93d7c5-db1a-415c-92e4-9ebec6cf195f"
-					(reference "R12")
+					(reference "R11")
 					(unit 1)
 				)
@@
 		(on_board yes)
 		(dnp no)
-		(property "Reference" "C21"
+		(property "Reference" "C20"
 			(at 82.296 130.302 90)
 			(effects
@@
 			(project "SUMEC_MK_V"
 				(path "/900bd7ac-cdf9-4a2f-8b1f-2c21e3760046/7b93d7c5-db1a-415c-92e4-9ebec6cf195f"
-					(reference "C21")
+					(reference "C20")
 					(unit 1)
 				)
@@
 		(on_board yes)
 		(dnp no)
-		(property "Reference" "U3"
+		(property "Reference" "U4"
 			(at 157.48 111.125 0)
 			(effects
@@
 			(project ""
 				(path "/900bd7ac-cdf9-4a2f-8b1f-2c21e3760046/7b93d7c5-db1a-415c-92e4-9ebec6cf195f"
-					(reference "U3")
+					(reference "U4")
 					(unit 1)
 				)
@@
 		(dnp no)
 		(fields_autoplaced yes)
-		(property "Reference" "#PWR056"
+		(property "Reference" "#PWR055"
 			(at 182.88 116.84 0)
 			(effects
@@
 			(project "SUMEC_MK_V"
 				(path "/900bd7ac-cdf9-4a2f-8b1f-2c21e3760046/7b93d7c5-db1a-415c-92e4-9ebec6cf195f"
-					(reference "#PWR056")
+					(reference "#PWR055")
 					(unit 1)
 				)
@@
 		(on_board yes)
 		(dnp no)
-		(property "Reference" "C22"
+		(property "Reference" "C21"
 			(at 187.96 46.99 90)
 			(effects
@@
 			(project "SUMEC_MK_V"
 				(path "/900bd7ac-cdf9-4a2f-8b1f-2c21e3760046/7b93d7c5-db1a-415c-92e4-9ebec6cf195f"
-					(reference "C22")
+					(reference "C21")
 					(unit 1)
 				)
@@
 		(on_board yes)
 		(dnp no)
-		(property "Reference" "#PWR055"
+		(property "Reference" "#PWR054"
 			(at 182.88 45.72 0)
 			(effects
@@
 			(project "SUMEC_MK_V"
 				(path "/900bd7ac-cdf9-4a2f-8b1f-2c21e3760046/7b93d7c5-db1a-415c-92e4-9ebec6cf195f"
-					(reference "#PWR055")
+					(reference "#PWR054")
 					(unit 1)
 				)
@@
 		(on_board yes)
 		(dnp no)
-		(property "Reference" "R13"
+		(property "Reference" "R12"
 			(at 222.885 83.82 0)
 			(effects
@@
 			(project "SUMEC_MK_V"
 				(path "/900bd7ac-cdf9-4a2f-8b1f-2c21e3760046/7b93d7c5-db1a-415c-92e4-9ebec6cf195f"
-					(reference "R13")
+					(reference "R12")
 					(unit 1)
 				)
@@
 		(on_board yes)
 		(dnp no)
-		(property "Reference" "#PWR058"
+		(property "Reference" "#PWR053"
 			(at 90.17 161.29 0)
 			(effects
@@
 			(project "SUMEC_MK_V"
 				(path "/900bd7ac-cdf9-4a2f-8b1f-2c21e3760046/7b93d7c5-db1a-415c-92e4-9ebec6cf195f"
-					(reference "#PWR058")
+					(reference "#PWR053")
 					(unit 1)
 				)
@@
 		(on_board yes)
 		(dnp no)
-		(property "Reference" "#PWR057"
+		(property "Reference" "#PWR052"
 			(at 90.17 137.16 0)
 			(effects
@@
 			(project "SUMEC_MK_V"
 				(path "/900bd7ac-cdf9-4a2f-8b1f-2c21e3760046/7b93d7c5-db1a-415c-92e4-9ebec6cf195f"
-					(reference "#PWR057")
+					(reference "#PWR052")
 					(unit 1)
 				)
@@
 		(dnp no)
 		(fields_autoplaced yes)
-		(property "Reference" "#PWR059"
+		(property "Reference" "#PWR056"
 			(at 198.12 58.42 0)
 			(effects
@@
 			(project "SUMEC_MK_V"
 				(path "/900bd7ac-cdf9-4a2f-8b1f-2c21e3760046/7b93d7c5-db1a-415c-92e4-9ebec6cf195f"
-					(reference "#PWR059")
+					(reference "#PWR056")
 					(unit 1)
 				)
@@
 		(on_board yes)
 		(dnp no)
-		(property "Reference" "C23"
+		(property "Reference" "C22"
 			(at 187.96 53.34 90)
 			(effects
@@
 			(project "SUMEC_MK_V"
 				(path "/900bd7ac-cdf9-4a2f-8b1f-2c21e3760046/7b93d7c5-db1a-415c-92e4-9ebec6cf195f"
-					(reference "C23")
-					(unit 1)
-				)
+					(reference "C22")
+					(unit 1)
+				)

Commit message: MK5 PCB rework
Parts:
- removed C20, C22: 100nF, Capacitor_SMD:C_0805_2012Metric_Pad1.18x1.45mm_HandSolder, symbol Device:C
- removed C21: 10uF, Capacitor_Tantalum_SMD:CP_EIA-3216-18_Kemet-A_Pad1.58x1.35mm_HandSolder, symbol Device:C_Polarized
- removed R11, R12: 10k, Resistor_SMD:R_0805_2012Metric_Pad1.20x1.40mm_HandSolder, symbol Device:R
- removed U3: 24CW1280T-I/OT, Package_TO_SOT_SMD:SOT-23-5, symbol Memory_EEPROM:24AA02-OT
- removed U4: ESP32-S3-WROOM-1, PCM_Espressif:ESP32-S3-WROOM-1, symbol sumec_sch_lib:ESP32-S3-WROOM-1_CUSTOM_made_by_bismarx
Connections:
- no-connect marks 7 -> 0
Other:
- note removed: "BAD PINOUT"
- note removed: "Default Configuration of Strapping Pins Strapping Pin Default Configuration Bit Value GPIO0 Pull-up 1 GPIO3 Floating - GPIO45 Pull-down 0 GPIO46 Pull-down 0"
- note removed: "EEPROM"
- note removed: "ESP32-S3 Datasheet"
- note removed: "ESP32-S3-WROOM1-N4"
- note removed: "GPIO0 has an internal pullup resistor, so if it is left unconnected then it will pull high."
- note removed: "GPIO0, GPIO45, and GPIO46 are connected to the chip's internal weak pull-up/pull-down resistors at chip reset. These resistors determine the default bit values of the strapping pins. Also, these resistors determine the bit values if the strapping pins are connected to an external high-impedance circuit."
- note removed: "I2C Addr.: 0x50"
- note removed: "Memory: 128kbit Ma freq.: 1MHz Vin: 1.6-5.5V Access time: 450ns Max supply curr.: 1mA"
- note removed: "NAME | GPIO | DESC. BOOT | 00 | BOOT mode, button LED_IO01 | 01 | LED, Indication, --debug BZ_IO02 | 02 | Buzzer, Indication --debug STRAP | 03 | STRAPPING PIN, DO NOT CONNECT BTN_IO04 | 04 | Button, INPUT_PULLPIT needed BTN_IO05 | 05 | Button, INPUT_PULLPIT needed PH_L | 06 | EN_L | 07 | EN_R | 08 | cSelect0 | 09 | cSelect1 | 10 | D_EXT1 | 11 | D_EXT2 | 12 | D_EXT3 | 13 | MODE_SW | 14 | RESET_SW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"
- note removed: "NO POL_L CONNECTED FIX TO IO35 NO ENCODERS CONNECTED FIX TO 4 AVAILABLE PINS"
- note removed: "SOME PINS ARE NOT CONNECTED IN SCHEMATIC"
- note removed: "Typically these can be used, but you need to make sure they are not in the wrong state during boot. gpio.0 Boot Mode. Weak pullup during reset. (Boot Mode 0=Boot from Flash, 1=Download) gpio.3 JTAG Mode. Weak pull down during reset. (JTAG Config) gpio.45 SPI voltage. Weak pull down during reset. (SPI Voltage 0=3.3v 1=1.8v) gpio.46 Boot mode. Weak pull down during reset. (Enabling/Disabling ROM Me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"
