File: main_hw/START_MODULE/START_MODULE.kicad_sch (KiCad schematic)
At the start: 12 parts, among them J1 Conn_01x03_Pin, J2 Conn_01x04_Pin, SW1 SW_Push, U1 ATtiny85-20S, U2 TSOP382xx

Commit message: PCB and 3d update
Changed lines of the file:
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@@
 (kicad_sch
-	(version 20231120)
+	(version 20250114)
 	(generator "eeschema")
-	(generator_version "8.0")
+	(generator_version "9.0")
 	(paper "A4")
+	(rectangle
+		(start 170.18 30.48)
+		(end 209.55 54.61)
+		(stroke
+			(width 0)
+			(type dash_dot)
+			(color 0 0 0 1)
+		)
+		(fill
+			(type none)
+		)
+	)
+	(rectangle
+		(start 123.19 30.48)
+		(end 162.56 54.61)
+		(stroke
+			(width 0)
+			(type dash_dot)
+			(color 0 0 0 1)
+		)
+		(fill
+			(type none)
+		)
+	)
+	(rectangle
+		(start 76.2 62.23)
+		(end 209.55 119.38)
+		(stroke
+			(width 0)
+			(type dash_dot)
+			(color 0 0 0 1)
+		)
+		(fill
+			(type none)
+		)
+	)
+	(rectangle
+		(start 76.2 30.48)
+		(end 115.57 54.61)
+		(stroke
+			(width 0)
+			(type dash_dot)
+			(color 0 0 0 1)
+		)
+		(fill
+			(type none)
+		)
+	)
+	(text "MCU"
+		(exclude_from_sim no)
+		(at 141.986 60.706 0)
+		(effects
+			(font
+				(face "Bahnschrift")
+				(size 4 4)
+				(thickness 0.8)
+				(bold yes)
+				(color 0 0 0 1)
+			)
+		)
+	)
+	(text "TSOP - IR RECIEVER"
+		(exclude_from_sim no)
+		(at 96.266 29.21 0)
+		(effects
+			(font
+				(face "Bahnschrift")
+				(size 3 3)
+				(thickness 0.8)
+				(bold yes)
+				(color 0 0 0 1)
+			)
+		)
+	)
+	(text "CONNECTORS"
+		(exclude_from_sim no)
+		(at 190.246 29.21 0)
+		(effects
+			(font
+				(face "Bahnschrift")
+				(size 3 3)
+				(thickness 0.6)
+				(bold yes)
+				(color 0 0 0 1)
+			)
+		)
+	)
+	(text "MCU RESET"
+		(exclude_from_sim no)
+		(at 142.748 29.21 0)
+		(effects
+			(font
+				(face "Bahnschrift")
+				(size 3 3)
+				(thickness 1)
+				(bold yes)
+				(color 0 0 0 1)
+			)
+		)
+	)
 	(junction
 		(at 115.57 80.01)
@@
 		)
 	)
-	(rectangle
-		(start 170.18 30.48)
-		(end 209.55 54.61)
-		(stroke
-			(width 0)
-			(type dash_dot)
-			(color 0 0 0 1)
-		)
-		(fill
-			(type none)
-		)
-	)
-	(rectangle
-		(start 123.19 30.48)
-		(end 162.56 54.61)
-		(stroke
-			(width 0)
-			(type dash_dot)
-			(color 0 0 0 1)
-		)
-		(fill
-			(type none)
-		)
-	)
-	(rectangle
-		(start 76.2 62.23)
-		(end 209.55 119.38)
-		(stroke
-			(width 0)
-			(type dash_dot)
-			(color 0 0 0 1)
-		)
-		(fill
-			(type none)
-		)
-	)
-	(rectangle
-		(start 76.2 30.48)
-		(end 115.57 54.61)
-		(stroke
-			(width 0)
-			(type dash_dot)
-			(color 0 0 0 1)
-		)
-		(fill
-			(type none)
-		)
-	)
 	(image
 		(at 158.75 137.16)
@@
 			"qAohhBBCCCGEKFIkUBVCCCGEEEIIUaRIoCqEEEIIIYQQokiRQFUIIYQQQgghRJEigaoQQgghhBBC"
 			"iCJFAlUhhBBCCCGEEEWKBKpCCCGEEEIIIYoUCVSFEEIIIYQQQhQpEqgKIYQQQgghhChSJFAVQggh"
-			"hBBCCFGk/A/J+il2alinwgAAAABJRU5ErkJggg=="
-		)
-	)
-	(text "MCU"
-		(exclude_from_sim no)
-		(at 141.986 60.706 0)
-		(effects
-			(font
-				(face "Bahnschrift")
-				(size 4 4)
-				(thickness 0.8)
-				(bold yes)
-				(color 0 0 0 1)
-			)
-		)
-	)
-	(text "TSOP - IR RECIEVER"
-		(exclude_from_sim no)
-		(at 96.266 29.21 0)
-		(effects
-			(font
-				(face "Bahnschrift")
-				(size 3 3)
-				(thickness 0.8)
-				(bold yes)
-				(color 0 0 0 1)
-			)
-		)
-	)
-	(text "CONNECTORS"
-		(exclude_from_sim no)
-		(at 190.246 29.21 0)
-		(effects
-			(font
-				(face "Bahnschrift")
-				(size 3 3)
-				(thickness 0.6)
-				(bold yes)
-				(color 0 0 0 1)
-			)
-		)
-	)
-	(text "MCU RESET"
-		(exclude_from_sim no)
-		(at 142.748 29.21 0)
-		(effects
-			(font
-				(face "Bahnschrift")
-				(size 3 3)
-				(thickness 1)
-				(bold yes)
-				(color 0 0 0 1)
-			)
+			"hBBCCFGk/A/J+il2alinwgAAAABJRU5ErkJgggAAAAAAAAAAAAAABwAAAAAAAAAAAAAAAAAAAAAA"
+			"AAAAAAAABAAAAAEAAAAAAAAAdwAAAL6QruQADgCAAG6GL+0BAAAAB5sv7QEAAABuhi/tAQAAAQAA"
+			"AAAAAAB8AAAAAAAAAAAAbgA2ADEALgBDAHUAAAAAAAAAAAAAAAcAAAAAAAAAAAAAAAAAAAAAAAAA"
+			"AAAAAAAAAAAAAAAAAAAAAAAAAAAAAAAAAAAAAAcAAAAAAAAAAAAAAAAAAAAAAAAAAAAAAAAAAAAB"
+			"AAAAAAAAAHwAAAC0kKTkAA8AgAMAAAAAAAAAAAAAAAAAAAAAAAAAAAAAAAAAAAAAAAAABwAAAAAA"
+			"AAAAAAAAAAAAAAAAAAAAAAAAAACIL+0BAAAAAAAAAAAAAAAAAAAAAAAABwAAAAAAAAAAAAAAAAAA"
+			"AAAAAAAAAAAADwAAAAEAAAAAAAAAAAAAAAAAAAAAAAAAAAAAAAAAAAABAAAAAAAAAAAAAAAAAAAA"
+			"SpGa5AAQAIABAAAAAAAAAAAAAAAAAAAAAAAAAAAAAAAAAAAAAAAAAAcAAAAAAAAAAAAAAAAAAAAA"
+			"AAAAAAAAAAAAbwBwAHAAZQByAAAAAAAAAAAAAAAAAAcAAAAAAAAAAAAAAAAAAAAAAAAAAAAAAAQA"
+			"AAABAAAAAAAAAAAAAAAAAAAAAAAAAAAAAAAAAAAAAQAAAAAAAAAAAAAAAAAAAECRkOQAEQCABQAA"
+			"AAAAAAAAAAAAAAAAAAAAAAAAAAAAAAAAAAAAAAAHAAAAAAAAAAAAAAAAAAAAAAAAAAAAAAAAAIgv"
+			"7QEAAAAAAAAAAAAAAAAAAAAAAAAHAAAAAAAAAAAAAAAAAAAAAAAAAAAAAAAHAAAAAQAAAAAAAAAA"
+			"AAAAAAAAAAAAAAAAAAAAAAAAAAEAAAAAAAAAAAAAAAAAAABWkYbkABIAgCQAewBLAEkAQwBBAEQA"
+			"OQBfADMARABNAE8ARABFAEwAXwBEAEkAUgB9AC8AQwBhAHAAYQBjAGkAdABvAHIAXwBTAE0ARAAu"
+			"ADMAZABzAGgAYQBwAGUAcwAvAEMAXwAwADgAMAA1AF8AMgAwADEAMgBNAGUAdAByAGkAYwAuAHcA"
+			"cgBsAAAAAAAAADMAOQAxADYAYQAAAAAAbJH85AATAIBgBpsv7QEAAOAImy/tAQAAwBSbL+0BAAAA"
+			"AAAAAAAAAHkAAAAAAAAAAABzAGUAcgAuADQAMgAAAAAAAAAAAAAABwAAAAAAAAAAAAAAAAAAAAAA"
+			"AAAAAAAAAAAAAAAAAAAAAAAAAAAAAAAAAAAAAAAABwAAAAAAAAAAAAAAAAAAAAAAAAAAAAAABAAA"
+			"AAEAAAAAAAAAeQAAAGKR8uQAFACAAG6GL+0BAA=="
 		)
 	)
 	(label "SCK"
 		(at 124.46 93.98 180)
-		(fields_autoplaced yes)
 		(effects
 			(font
@@
 	(label "MISO"
 		(at 185.42 49.53 0)
-		(fields_autoplaced yes)
 		(effects
 			(font
@@
 	(label "~{CS}"
 		(at 132.08 46.99 0)
-		(fields_autoplaced yes)
 		(effects
 			(font
@@
 	(label "MOSI"
 		(at 147.32 80.01 0)
-		(fields_autoplaced yes)
 		(effects
 			(font
@@
 	(label "~{CS}"
 		(at 132.08 38.1 0)
-		(fields_autoplaced yes)
 		(effects
 			(font
@@
 	(label "~{CS}"
 		(at 185.42 44.45 0)
-		(fields_autoplaced yes)
 		(effects
 			(font
@@
 	(label "MISO"
 		(at 147.32 88.9 0)
-		(fields_autoplaced yes)
 		(effects
 			(font
@@
 	(label "MISO"
 		(at 124.46 91.44 180)
-		(fields_autoplaced yes)
 		(effects
 			(font
@@
 	(label "SCK"
 		(at 185.42 46.99 0)
-		(fields_autoplaced yes)
 		(effects
 			(font
@@
 	(label "~{CS}"
 		(at 124.46 101.6 180)
-		(fields_autoplaced yes)
 		(effects
 			(font
@@
 	(label "MOSI"
 		(at 185.42 52.07 0)
-		(fields_autoplaced yes)
 		(effects
 			(font
@@
 	(label "MOSI"
 		(at 124.46 88.9 180)
-		(fields_autoplaced yes)
 		(effects
 			(font
@@
 		)
 	)
+	(embedded_fonts no)
 )
