File: main_hw/START_MODULE/START_MODULE.kicad_pcb (KiCad board)
At the start: 2 copper layers, 18.5 x 13 mm, 12 parts, among them J1 Conn_01x03_Pin, J2 Conn_01x04_Pin, SW1 SW_Push, U1 ATtiny85-20S, U2 TSOP382xx

Commit message: MK5 new update of the PCB
Parts:
- J1: footprint Connector_PinHeader_2.54mm:PinHeader_1x03_P2.54mm_Vertical -> Connector_PinHeader_2.54mm:PinHeader_1x03_P2.54mm_Horizontal
