File: main_hw/QRE_MINIBOARD_V2/QRE_MiniBoardV2.kicad_pcb (KiCad board)
At the start: 2 copper layers, 97 x 16.5 mm, 11 parts, among them J1 Conn_01x04_Pin, U1 QRE1113, U2 QRE1113

Commit message: silkscreen
Other:
- board text added: "made by: bismarx"
