File: main_hw/SUMEC_MK_V_Pro/SUMEC_MK_V_Pro.kicad_sch (KiCad schematic)
At the start: 134 parts, among them J1 XT30PW-M, J10 Conn_01x03_Pin, J11 Conn_01x03_Pin, J12 Conn_01x06_Pin, J13 Conn_01x03_Pin, J2 Conn_01x06_Socket, J3 Conn_01x06_Socket, J4 USB_C, J5 Conn_01x03_Pin, J6 Conn_01x04_Pin, J7 Conn_01x03_Pin, J8 Conn_01x03_Pin, J9 Conn_01x03_Pin, Q1 PMOS, SW1 SW_DPDT_x2, SW2 RST, SW3 RESET, SW4 BOOT, SW5 BOOT, SW6 BOOT, U1 INA226, U2 DRV8874PWPR, U3 DRV8874PWPR, U4 AP62300Z6, U5 TPS565242DRLR, U6 USBLC6-2SC6, U7 BNO055, U8 ESP32-S3-WROOM-1, U9 24CW1280T-I/OT, Y1 32.768k

Commit message: Final update for MK Pro
PCB, schematic update, IMU software
Other:
- note removed: "BNO055: 0x28 EEPROM: 0x50 FUSB302 0x25 BQ2589: 0x6A GNSS: 0x3A"
Changed lines of the file:
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@@
-		)
-	)
-	(text "BNO055:   0x28\nEEPROM:  0x50\nFUSB302  0x25\nBQ2589:   0x6A\nGNSS:      0x3A"
-		(exclude_from_sim no)
-		(at 327.025 110.49 0)
-		(effects
-			(font
-				(face "Bahnschrift")
-				(size 2 2)
-				(color 0 0 0 1)
-			)
-			(justify left bottom)
 		)
 	)

Commit message: Prepare for release
Other:
- note added: "0x28/0x29 - BNO055 0x40 - INA226 0x50 - 24CW1280T 0xXX - TF-LUNA"
- note added: "BUG: NOT ADC"
- note added: "I2C Addr.: 0x28 I2C Addr.: 0x29 when COM3 tied to 3V3"
- note removed: "1. Bigger inductor for 3.3V 2. 3. 4. 5. 6. 7."
- note removed: "CHANGES:"
- note removed: "I2C Addr.: 0x28"
- note removed: "I2C Addr.: 0x29 when COM3 tied to 3V3"
- moved on the sheet: BZ1, C1, C10, C11, C12, C13, C14, C15, C16, C17, C18, C19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
